File: SOC DISPLAY.kicad_pcb (KiCad board)
At the start: 2 copper layers, 58 parts, among them IC1 CM BLE, IC2 LM5164QDDATQ1, J1 Conn_01x05_Socket, J2 OLED, J3 PRG, J4 Conn_01x02_Socket, Q1 NDT3055L, U1 STM32G0B1CBTx, U2 MAX485E, U3 TJA1051T-3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

Commit message: new change
Parts:
- moved J2 15.9 mm to (107.5, 44.5)
Changed lines of the file:
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@@
     (property "ki_keywords" "mounting hole")
     (attr exclude_from_pos_files)
-    (fp_text reference "H1" (at 0 -3.25) (layer "F.SilkS")
+    (fp_text reference "H1" (at -6.977 -17.517) (layer "F.SilkS")
         (effects (font (size 1 1) (thickness 0.15)))
     )
@@
   )
   (footprint "TerminalBlock:TerminalBlock_bornier-4_P5.08mm" (layer "F.Cu")
-    (at 114.435 58.735)
+    (at 107.458 44.468)
     (descr "simple 4-pin terminal block, pitch 5.08mm, revamped version of bornier4")
     (tags "terminal block bornier4")

Commit message: changes
Parts:
- removed R22: 120k, Resistor_SMD:R_0603_1608Metric_Pad0.98x0.95mm_HandSolder
- removed R23, R24: 453k ohm, Resistor_SMD:R_0603_1608Metric_Pad0.98x0.95mm_HandSolder
- added 100k1: R24, Resistor_SMD:R_0603_1608Metric_Pad0.98x0.95mm_HandSolder, F.Cu at (171.2, 65.2)
- added 1M1: R22, Resistor_SMD:R_0603_1608Metric_Pad0.98x0.95mm_HandSolder, F.Cu at (171.2, 67.7)
- added 332k1: R23, Resistor_SMD:R_0603_1608Metric_Pad0.98x0.95mm_HandSolder, F.Cu at (171.2, 70.2)
- added C11: 22UF, Capacitor_SMD:C_1206_3216Metric_Pad1.33x1.80mm_HandSolder, F.Cu at (181.2, 74.5)
- added C12: 10nf, Capacitor_SMD:C_0805_2012Metric_Pad1.18x1.45mm_HandSolder, F.Cu at (175.8, 74.4)
- added C13: 2.2uf, Capacitor_SMD:C_0805_2012Metric_Pad1.18x1.45mm_HandSolder, F.Cu at (175.8, 77.4)
- added E1: LI0603G121R-10, LI0603G121R-10.kicad_mod files:FB_LI0603G121R-10, F.Cu at (178.7, 68.6)
- added R26: 180k ohm, Resistor_SMD:R_0603_1608Metric_Pad0.98x0.95mm_HandSolder, F.Cu at (171.2, 72.7)
- added R27: 20k ohm, Resistor_SMD:R_0603_1608Metric_Pad0.98x0.95mm_HandSolder, F.Cu at (171.2, 75.2)
- C1: value 2.2uf -> 1uF; footprint Capacitor_SMD:C_1210_3225Metric_Pad1.33x2.70mm_HandSolder -> Capacitor_SMD:C_0805_2012Metric_Pad1.18x1.45mm_HandSolder
- C2: value 0.1uf -> 100nF
- C3: value 2.2nf -> 100nF; footprint Capacitor_SMD:C_0603_1608Metric_Pad1.08x0.95mm_HandSolder -> Capacitor_SMD:C_0805_2012Metric_Pad1.18x1.45mm_HandSolder
- C5: value 56pF -> 2.2uF
- C6: value 0.1uf -> 2.2nf; footprint Capacitor_SMD:C_0805_2012Metric_Pad1.18x1.45mm_HandSolder -> Capacitor_SMD:C_0603_1608Metric_Pad1.08x0.95mm_HandSolder
- C7: value 3.3nf -> 56pF; footprint Capacitor_SMD:C_0805_2012Metric_Pad1.18x1.45mm_HandSolder -> Capacitor_SMD:C_0402_1005Metric_Pad0.74x0.62mm_HandSolder
- C8: value 0.1uf -> 1uf
- C9: value 22UF -> 2200pf; footprint Capacitor_SMD:C_1206_3216Metric_Pad1.33x1.80mm_HandSolder -> Capacitor_SMD:C_0805_2012Metric_Pad1.18x1.45mm_HandSolder
- L2: value 68uH -> 100uH
- R11: value 0R -> 120R
- R12, R13: value 0R -> 100E
- R14: value 120R -> 0R
- R15, R6: value 100E -> 100k
- R16: value 100E -> 10k
- R17: value 0R -> 56k
- R18: value 100k -> 120R
- R19: value 10k -> 3M
- R20: value 100k ohm -> 100E
- R21: value 56k -> 0R
- R25: value 49.9k ohm -> 698k ohm
- R5: value 3M -> 100k
- R7, R8: value 100k -> 0R
Connections:
- C1 pad 1: 100V -> Vdd
- C2 pad 1: VBST -> Vdd
- C2 pad 2: SW2 -> GND
- C3 pad 1: Net-(IC2-SW) -> Vdd
- C3 pad 2: Net-(IC2-BST) -> GND
- C4 pad 1: GND -> VBST
- C4 pad 2: /3V3 -> SW2
- C5 pad 1: Net-(IC2-FB) -> Net-(IC2-GND)
- C5 pad 2: Net-(C5-Pad2) -> 100V
- C6 pad 1: GND -> Net-(IC2-SW)
- C6 pad 2: /3V3 -> Net-(IC2-BST)
- C7 pad 1: Net-(C5-Pad2) -> Net-(IC2-FB)
- C7 pad 2: /12V -> Net-(C7-Pad2)
- C8 pad 1: /3V3 -> 5V
- C9 pad 1: /12V -> Net-(C7-Pad2)
- C9 pad 2: GND -> /12V
- IC1 pad 18: /3V3 -> Vdd
- IC1 pad 19: /3V3 -> Vdd
- IC1 pad 20: /3V3 -> Vdd
- IC2 pad 1: GND -> Net-(IC2-GND)
- IC2 pad 3: 100V -> Net-(IC2-EN/UVLO)
- R1 pad 1: /3V3 -> Vdd
- R10 pad 1: 5V -> SDA
- R10 pad 2: Net-(BZ1--) -> Net-(J1-Pin_3)
- R11 pad 1: SCK -> Net-(J4-Pin_2)
- R11 pad 2: Net-(J1-Pin_2) -> Net-(J4-Pin_1)
- R12 pad 1: Net-(J1-Pin_2) -> SCK
- R12 pad 2: L -> SCL
- R13 pad 1: 5V -> SDA1
- R13 pad 2: Net-(J1-Pin_3) -> SDA
- R14 pad 1: Net-(J4-Pin_2) -> Net-(J1-Pin_3)
- R14 pad 2: Net-(J4-Pin_1) -> H
- R15 pad 1: SCK -> Net-(U3-S)
- R15 pad 2: SCL -> GND
- R16 pad 1: SDA1 -> GND
- R16 pad 2: SDA -> VFB
- R17 pad 1: Net-(J1-Pin_3) -> VFB
- R17 pad 2: H -> 5V
- R18 pad 1: Net-(U3-S) -> L
- R18 pad 2: GND -> H
- R19 pad 1: GND -> Net-(D1-K)
- R19 pad 2: VFB -> GND
- R20 pad 1: Net-(IC2-RON) -> PA3
- R20 pad 2: GND -> Net-(D1-K)
- R21 pad 1: VFB -> 5V
- R21 pad 2: 5V -> Net-(BZ1--)
- R25 pad 1: Net-(IC2-FB) -> Net-(IC2-SW)
- R25 pad 2: GND -> Net-(C7-Pad2)
- R5 pad 1: Net-(D1-K) -> Vdd
- R5 pad 2: GND -> SCL
- R6 pad 1: PA3 -> Vdd
- R6 pad 2: Net-(D1-K) -> SDA
- R7 pad 1: /3V3 -> 5V
- R7 pad 2: SCL -> Net-(J1-Pin_1)
- R8 pad 1: /3V3 -> SCK
- R8 pad 2: SDA -> Net-(J1-Pin_2)
- R9 pad 1: SDA -> Net-(J1-Pin_2)
- R9 pad 2: Net-(J1-Pin_1) -> L
- U1 pad 4: /3V3 -> Vdd
- U1 pad 5: /3V3 -> Vdd
- U1 pad 6: /3V3 -> Vdd
- U3 pad 5: /3V3 -> Vdd
- U5 pad 4: unconnected-(U5-BP-Pad4) -> Net-(U5-BP)
- U5 pad 5: /3V3 -> Vdd

Commit message: 3V3
Parts:
- R22: renamed from 1M1; value R22 -> 1M
- R23: renamed from 332k1; value R23 -> 332k
- R24: renamed from 100k1; value R24 -> 100K
- moved C9 88.8 mm to (186.2, 52.0)
- moved C10 80.3 mm to (186.9, 56.9)
- moved L1 75.8 mm to (182.6, 62.2), turned to 180 degrees
- moved L2 74.2 mm to (186.2, 50.0)
- moved C5 72.7 mm to (172.8, 51.2), turned to -90 degrees
- moved C7 59.7 mm to (182.2, 53.6)
- moved C6 58.8 mm to (181.8, 51.5), turned to -90 degrees
- moved R25 56.2 mm to (183.3, 51.4), turned to -90 degrees
- moved R17 52.7 mm to (183.0, 60.5), turned to 180 degrees
- moved R16 52.2 mm to (183.0, 58.9)
- moved C4 51.9 mm to (186.9, 63.0)
- moved F1 51.3 mm to (171.6, 51.2), turned to -90 degrees
- moved U4 50.9 mm to (186.8, 60.0), turned to 180 degrees
- moved U5 43.7 mm to (179.2, 59.9), turned to 180 degrees
- moved C13 41.1 mm to (216.9, 77.7)
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Other:
- board outline added: 41.1 x 39.4 mm

Commit message: chanses made
Parts:
- removed R22: 1M, Resistor_SMD:R_0603_1608Metric_Pad0.98x0.95mm_HandSolder
- removed R23: 332k, Resistor_SMD:R_0603_1608Metric_Pad0.98x0.95mm_HandSolder
- removed R24: 100K, Resistor_SMD:R_0603_1608Metric_Pad0.98x0.95mm_HandSolder
- added 100k1: R24, Resistor_SMD:R_0603_1608Metric_Pad0.98x0.95mm_HandSolder, F.Cu at (185.9, 71.4)
- added 1M1: R22, Resistor_SMD:R_0603_1608Metric_Pad0.98x0.95mm_HandSolder, F.Cu at (185.9, 73.9)
- added 332k1: R23, Resistor_SMD:R_0603_1608Metric_Pad0.98x0.95mm_HandSolder, F.Cu at (185.9, 76.5)
Connections:
- net Vdd renamed /3V3

Commit message: placing
Parts:
- Q1: moved to B.Cu
- R22: renamed from 1M1; value R22 -> 1M
- R24: renamed from 100k1; value R24 -> 100K
- moved J4 93.2 mm to (200.4, 50.5), turned to 90 degrees
- moved J3 77.3 mm to (200.4, 66.3), turned to 90 degrees
- moved C1 74.6 mm to (180.3, 49.6), turned to 90 degrees
- moved H4 73.2 mm to (201.9, 75.9)
- moved R11 73.1 mm to (195.6, 51.6), turned to -90 degrees
- moved U1 72.9 mm to (174.1, 51.5), turned to 180 degrees
- moved H2 68.5 mm to (201.9, 40.1)
- moved C8 67.1 mm to (188.7, 52.3)
- moved R3 65.7 mm to (180.7, 46.7)
- moved R1 62.4 mm to (182.1, 49.7), turned to 90 degrees
- moved R5 60.7 mm to (173.8, 59.9)
- moved U2 60.1 mm to (193.4, 57.1), turned to 90 degrees
- moved R19 59.6 mm to (189.5, 63.0)
- moved R9 58.3 mm to (182.1, 52.9), turned to -90 degrees
- moved D1 57.7 mm to (180.7, 63.0), turned to 180 degrees
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- renumbered H5 to H1, H6 to H2, H1 to H4, H4 to H5, H2 to H6, 332k1 to R23
Routing:
- net /12V: track 0.00 -> 15.9 mm
- net Net-(IC2-SW): track 0.00 -> 5.44 mm
- net 100V: track 0.00 -> 4.90 mm
- net Net-(IC2-FB): track 0.00 -> 4.81 mm
- net 5V: track 0.00 -> 3.68 mm
- net Net-(IC2-EN/UVLO): track 0.00 -> 3.63 mm
- net Net-(C7-Pad2): track 0.00 -> 3.46 mm
- net VBST: track 0.00 -> 2.11 mm
- net Net-(IC2-BST): track 0.00 -> 2.04 mm
- net /3V3: track 0.00 -> 1.97 mm
- net Net-(IC2-RON): track 0.00 -> 1.91 mm
- net H: track 0.00 -> 1.82 mm
- net Net-(IC2-GND): track 0.00 -> 1.74 mm
- net L: track 0.00 -> 1.48 mm
- net /RX: track 0.00 -> 1.33 mm
Other:
- board size 41.1 x 39.4 mm -> 48.8 x 41.1 mm

Commit message: frst
Parts:
- added 100k1: R24, Resistor_SMD:R_0603_1608Metric_Pad0.98x0.95mm_HandSolder, F.Cu at (215.6, 46.9)
- added 1M1: R22, Resistor_SMD:R_0603_1608Metric_Pad0.98x0.95mm_HandSolder, F.Cu at (215.6, 49.4)
- added 332k1: R23, Resistor_SMD:R_0603_1608Metric_Pad0.98x0.95mm_HandSolder, F.Cu at (215.6, 51.9)
- added J5: Conn_01x02_Socket, TerminalBlock:TerminalBlock_bornier-2_P5.08mm, F.Cu at (221.0, 50.2)
- added R28: 180k ohm, Resistor_SMD:R_0603_1608Metric_Pad0.98x0.95mm_HandSolder, F.Cu at (215.6, 54.5)
- added R29: 20k ohm, Resistor_SMD:R_0603_1608Metric_Pad0.98x0.95mm_HandSolder, F.Cu at (215.6, 57.0)
- J1: value Conn_01x05_Socket -> PRG; footprint Connector_JST:JST_PH_S5B-PH-K_1x05_P2.00mm_Horizontal -> TerminalBlock:TerminalBlock_bornier-3_P5.08mm
- J2: value OLED -> Conn_01x05_Socket; footprint TerminalBlock:TerminalBlock_bornier-4_P5.08mm -> Connector_JST:JST_PH_S5B-PH-K_1x05_P2.00mm_Horizontal
- J3: value PRG -> OLED; footprint TerminalBlock:TerminalBlock_bornier-3_P5.08mm -> TerminalBlock:TerminalBlock_bornier-4_P5.08mm
- J4: value Conn_01x02_Socket -> OLED; footprint TerminalBlock:TerminalBlock_bornier-2_P5.08mm -> TerminalBlock:TerminalBlock_bornier-4_P5.08mm
- R10, R14, R9: value 0R -> 100k
- R11: value 120R -> 100E
- R13, R20: value 100E -> 100k
- R15: value 100k -> 100E
- R16: value 10k -> 100E
- R17: value 56k -> 0R
- R19: value 3M -> 0R
- R21: value 0R -> 10k
- R22: value 1M -> 56k
- R23: value R23 -> 120R
- R24: value 100K -> 3M
- R25: value 698k ohm -> 100E
- R26: value 180k ohm -> 0R
- R27: value 20k ohm -> 698k ohm
- R5, R6: value 100k -> 0R
Connections:
- F1 pad 1: Net-(J1-Pin_1) -> Net-(J2-Pin_1)
- J1 pad 1: Net-(J1-Pin_1) -> SWCLK
- J1 pad 2: Net-(J1-Pin_2) -> SWDIO
- J1 pad 3: Net-(J1-Pin_3) -> GND
- J2 pad 1: 5V -> Net-(J2-Pin_1)
- J2 pad 2: SDA1 -> Net-(J2-Pin_2)
- J2 pad 3: SCK -> Net-(J2-Pin_3)
- J3 pad 1: SWCLK -> 5V
- J3 pad 2: SWDIO -> SDA_2
- J3 pad 3: GND -> SCK_2
- J4 pad 1: Net-(J4-Pin_1) -> 5V
- J4 pad 2: Net-(J4-Pin_2) -> SDA1
- R10 pad 1: SDA -> /3V3
- R10 pad 2: Net-(J1-Pin_3) -> SDA_PB7
- R11 pad 1: Net-(J4-Pin_2) -> SCK_2
- R11 pad 2: Net-(J4-Pin_1) -> SCL_PB4
- R12 pad 1: SCK -> SDA_2
- R12 pad 2: SCL -> SDA_PB7
- R13 pad 1: SDA1 -> /3V3
- R13 pad 2: SDA -> SCL_PB3
- R14 pad 1: Net-(J1-Pin_3) -> /3V3
- R14 pad 2: H -> SDA_PB4
- R15 pad 1: Net-(U3-S) -> SCK
- R15 pad 2: GND -> SCL_PB6
- R16 pad 1: GND -> SDA1
- R16 pad 2: VFB -> SDA_PB7
- R17 pad 1: VFB -> SDA_PB7
- R17 pad 2: 5V -> Net-(J2-Pin_3)
- R18 pad 1: L -> Net-(J5-Pin_2)
- R18 pad 2: H -> Net-(J5-Pin_1)
- R19 pad 1: Net-(D1-K) -> Net-(J2-Pin_3)
- R19 pad 2: GND -> H
- R20 pad 1: PA3 -> Net-(U3-S)
- R20 pad 2: Net-(D1-K) -> GND
- R21 pad 1: 5V -> GND
- R21 pad 2: Net-(BZ1--) -> VFB
- R22 pad 1: 100V -> VFB
- R22 pad 2: Net-(IC2-EN/UVLO) -> 5V
- R23 pad 1: Net-(IC2-EN/UVLO) -> L
- R23 pad 2: GND -> H
- R24 pad 1: Net-(IC2-RON) -> Net-(D1-K)
- R25 pad 1: Net-(IC2-SW) -> PA3
- R25 pad 2: Net-(C7-Pad2) -> Net-(D1-K)
- R26 pad 1: /12V -> 5V
- R26 pad 2: Net-(IC2-FB) -> Net-(BZ1--)
- R27 pad 1: Net-(IC2-FB) -> Net-(IC2-SW)
- R27 pad 2: GND -> Net-(C7-Pad2)
- R5 pad 1: /3V3 -> 5V
- R5 pad 2: SCL -> Net-(J2-Pin_1)
- R6 pad 1: /3V3 -> /12V
- R6 pad 2: SDA -> Net-(J2-Pin_1)
- R7 pad 1: 5V -> SCK
- R7 pad 2: Net-(J1-Pin_1) -> Net-(J2-Pin_2)
- R8 pad 1: SCK -> Net-(J2-Pin_2)
- R8 pad 2: Net-(J1-Pin_2) -> L
- R9 pad 1: Net-(J1-Pin_2) -> /3V3
- R9 pad 2: L -> SCL_PB6
- U1 pad 42: unconnected-(U1-PB3-Pad42) ->  SCL_PB3
- U1 pad 43: unconnected-(U1-PB4-Pad43) -> SDA_PB4
- U1 pad 45: SCL -> SCL_PB6
- U1 pad 46: SDA -> SDA_PB7
- U2 pad 6: Net-(J4-Pin_2) -> Net-(J5-Pin_2)
- U2 pad 7: Net-(J4-Pin_1) -> Net-(J5-Pin_1)
Routing:
- net Net-(J2-Pin_3): track 0.00 -> 0.53 mm
- net 5V: track 3.68 -> 3.15 mm

Commit message: Matic
Parts:
- R22: renamed from 1M1; value R22 -> 1M1
- R23: renamed from 332k1; value R23 -> 332K
- R24: renamed from 100k1; value R24 -> 100K
- moved R23 100.6 mm to (115.0, 49.8), turned to 180 degrees
- moved R22 99.8 mm to (115.8, 47.4), turned to -90 degrees
- moved R24 97.3 mm to (118.4, 50.0)
- moved R11 90.2 mm to (105.9, 61.2)
- moved R29 89.9 mm to (125.8, 50.7)
- moved R28 89.8 mm to (125.9, 49.1), turned to 180 degrees
- moved R17 86.5 mm to (103.3, 62.2)
- moved R16 86.4 mm to (103.3, 60.2)
- moved R20 76.6 mm to (109.1, 71.7), turned to 0 degrees
- moved R14 71.4 mm to (110.7, 61.3)
- moved U3 70.6 mm to (116.4, 55.5)
- moved R9 70.4 mm to (112.3, 61.3), turned to 90 degrees
- moved C3 69.5 mm to (111.5, 49.3), turned to 90 degrees
- moved R13 69.2 mm to (108.5, 61.4), turned to -90 degrees
- moved R4 69.1 mm to (100.6, 57.1)
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Routing:
- net /12V: track 15.9 -> 0.00 mm
- net Net-(IC2-SW): track 5.44 -> 0.00 mm
- net 100V: track 4.90 -> 0.00 mm
- net Net-(IC2-FB): track 4.81 -> 0.00 mm
- net Net-(IC2-EN/UVLO): track 3.63 -> 0.00 mm
- net Net-(C7-Pad2): track 3.46 -> 0.00 mm
- net 5V: track 3.15 -> 0.00 mm
- net VBST: track 2.11 -> 0.00 mm
- net Net-(IC2-BST): track 2.04 -> 0.00 mm
- net Net-(IC2-RON): track 1.91 -> 0.00 mm
- net H: track 1.82 -> 0.00 mm
- net Net-(IC2-GND): track 1.74 -> 0.00 mm
- net L: track 1.48 -> 0.00 mm
- net /3V3: track 1.97 -> 0.61 mm
- net /RX: track 1.33 -> 0.00 mm

Commit message: chull
Parts:
- added 100k1: R24, Resistor_SMD:R_0603_1608Metric_Pad0.98x0.95mm_HandSolder, F.Cu at (144.6, 28.1)
- added 1M1: R22, Resistor_SMD:R_0603_1608Metric_Pad0.98x0.95mm_HandSolder, F.Cu at (144.6, 30.6)
- added 332k1: R23, Resistor_SMD:R_0603_1608Metric_Pad0.98x0.95mm_HandSolder, F.Cu at (144.6, 33.1)
- R22: value 1M1 -> 56k
- R23: value 332K -> 120R
- R24: value 100K -> 3M
Connections:
- R11 pad 2: SCL_PB4 -> SCL_PB3
- R12 pad 2: SDA_PB7 -> SDA_PB4
- R22 pad 1: 100V -> VFB
- R22 pad 2: Net-(IC2-EN/UVLO) -> 5V
- R23 pad 1: Net-(IC2-EN/UVLO) -> L
- R23 pad 2: GND -> H
- R24 pad 1: Net-(IC2-RON) -> Net-(D1-K)
