File: SOC DISPLAY.kicad_pcb (KiCad board)
At the start: 2 copper layers, 48.8 x 41.1 mm, 70 parts, among them IC1 CM BLE, IC2 LM5164QDDATQ1, J1 PRG, J2 Conn_01x05_Socket, J3 OLED, J4 OLED, J5 Conn_01x02_Socket, Q1 NDT3055L, U1 STM32G0B1CBTx, U2 MAX485E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

Commit message: Done
Parts:
- Q1: moved to B.Cu
- moved R1 72.4 mm to (182.1, 49.7)
- moved E1 64.6 mm to (122.9, 69.8)
- moved R5 49.6 mm to (125.8, 52.1)
- moved R6 34.0 mm to (132.1, 45.7), turned to -90 degrees
- moved R7 22.0 mm to (136.0, 67.6)
- moved Q1 10.1 mm to (183.3, 65.5), turned to 180 degrees
- moved R10 8.43 mm to (108.1, 62.2), turned to 0 degrees
- moved R17 7.87 mm to (111.0, 60.7), turned to -90 degrees
- moved R13 6.86 mm to (101.6, 61.6)
- moved R16 6.26 mm to (109.5, 59.3), turned to 90 degrees
- moved R9 6.19 mm to (106.4, 59.3)
- moved R12 6.17 mm to (108.0, 59.3)
- moved R14 6.17 mm to (104.9, 59.3)
- moved R11 5.95 mm to (102.4, 65.9)
- moved R23 1.69 mm to (111.8, 56.7)
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Routing:
- net Net-(J2-Pin_3): track 0.53 -> 0.00 mm

Commit message: Placing Soc
Parts:
- Q1: moved to F.Cu
- moved J4 110.5 mm to (92.5, 73.9)
- moved J5 92.6 mm to (132.6, 77.7), turned to 180 degrees
- moved R15 81.9 mm to (102.7, 61.0)
- moved J1 80.7 mm to (92.5, 53.1), turned to 90 degrees
- moved J3 77.5 mm to (127.8, 39.4), turned to 180 degrees
- moved R1 72.6 mm to (109.5, 50.3)
- moved R3 71.7 mm to (109.0, 47.2)
- moved BZ1 71.1 mm to (114.3, 73.2)
- moved H1 67.4 mm to (90.9, 37.6)
- moved IC1 67.2 mm to (103.6, 71.4)
- moved H3 67.1 mm to (91.2, 79.2)
- moved D1 66.8 mm to (114.0, 64.8)
- moved Q1 63.2 mm to (120.1, 62.2), turned to 0 degrees
- moved J2 57.0 mm to (107.2, 42.2), turned to 180 degrees
- moved R26 41.2 mm to (118.5, 51.8)
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Routing:
- net /3V3: track 0.61 -> 0.00 mm
Other:
- board size 48.8 x 41.1 mm -> 47.2 x 46.7 mm
