File: SOC DISPLAY.kicad_pcb (KiCad board)
At the start: 2 copper layers, 47.2 x 46.7 mm, 70 parts, among them IC1 CM BLE, IC2 LM5164QDDATQ1, J1 PRG, J2 Conn_01x05_Socket, J3 OLED, J4 OLED, J5 Conn_01x02_Socket, Q1 NDT3055L, U1 STM32G0B1CBTx, U2 MAX485E, U3 TJA1051T-3, U4 TPS563200, U5 LP2985-3.3

Commit message: giga
Parts:
- added C14: 22uF, Capacitor_SMD:C_1206_3216Metric_Pad1.33x1.80mm_HandSolder, F.Cu at (195.6, 48.8)
- added C15: 22uF, Capacitor_SMD:C_1206_3216Metric_Pad1.33x1.80mm_HandSolder, F.Cu at (195.6, 52.1)
- added C16: 22uF, Capacitor_SMD:C_1206_3216Metric_Pad1.33x1.80mm_HandSolder, F.Cu at (195.6, 55.5)
- added C17: 22uF, Capacitor_SMD:C_1206_3216Metric_Pad1.33x1.80mm_HandSolder, F.Cu at (195.6, 58.8)
- added J6: Conn_01x02_Pin, TerminalBlock:TerminalBlock_bornier-2_P5.08mm, F.Cu at (184.2, 51.6)
- added J7: Conn_01x02_Pin, TerminalBlock:TerminalBlock_bornier-2_P5.08mm, F.Cu at (184.2, 60.7)
- added R30: 3M, Resistor_SMD:R_0603_1608Metric_Pad0.98x0.95mm_HandSolder, F.Cu at (202.7, 48.4)
- added R31: 100E, Resistor_SMD:R_0603_1608Metric_Pad0.98x0.95mm_HandSolder, F.Cu at (202.7, 50.9)
- added R32: 0R, Resistor_SMD:R_0603_1608Metric_Pad0.98x0.95mm_HandSolder, F.Cu at (202.7, 53.4)
- added R33: 100k, Resistor_SMD:R_0603_1608Metric_Pad0.98x0.95mm_HandSolder, F.Cu at (202.7, 57.9)
- added R34: 120R, Resistor_SMD:R_0603_1608Metric_Pad0.98x0.95mm_HandSolder, F.Cu at (202.7, 60.4)
- added R35: 10k, Resistor_SMD:R_0603_1608Metric_Pad0.98x0.95mm_HandSolder, F.Cu at (178.8, 48.4)
- added R36: 10k, Resistor_SMD:R_0603_1608Metric_Pad0.98x0.95mm_HandSolder, F.Cu at (178.8, 50.9)
- added R37: 100R, Resistor_SMD:R_0603_1608Metric_Pad0.98x0.95mm_HandSolder, F.Cu at (178.8, 53.4)
- added R38: 16.2M, Resistor_SMD:R_0603_1608Metric_Pad0.98x0.95mm_HandSolder, F.Cu at (178.8, 55.9)
- added R39: 100R, Resistor_SMD:R_0603_1608Metric_Pad0.98x0.95mm_HandSolder, F.Cu at (178.8, 58.4)
- added R40: 10k, Resistor_SMD:R_0603_1608Metric_Pad0.98x0.95mm_HandSolder, F.Cu at (178.8, 60.9)
- added R41: 10k, Resistor_SMD:R_0603_1608Metric_Pad0.98x0.95mm_HandSolder, F.Cu at (178.8, 63.4)
- added R42: 10k, Resistor_SMD:R_0603_1608Metric_Pad0.98x0.95mm_HandSolder, F.Cu at (178.8, 65.9)
- added U6: INA228AQDGSRQ1, Package_SO:VSSOP-10_3x3mm_P0.5mm, F.Cu at (184.7, 67.5)
- C1: value 1uF -> 0.1uf; footprint Capacitor_SMD:C_0805_2012Metric_Pad1.18x1.45mm_HandSolder -> Capacitor_SMD:C_0603_1608Metric_Pad1.08x0.95mm_HandSolder
- C11: value 22UF -> 1uF; footprint Capacitor_SMD:C_1206_3216Metric_Pad1.33x1.80mm_HandSolder -> Capacitor_SMD:C_0603_1608Metric_Pad1.08x0.95mm_HandSolder
- C12: value 10nf -> 100nF; footprint Capacitor_SMD:C_0805_2012Metric_Pad1.18x1.45mm_HandSolder -> Capacitor_SMD:C_0603_1608Metric_Pad1.08x0.95mm_HandSolder
- C13: value 2.2uf -> 100nF; footprint Capacitor_SMD:C_0805_2012Metric_Pad1.18x1.45mm_HandSolder -> Capacitor_SMD:C_0603_1608Metric_Pad1.08x0.95mm_HandSolder
- C2: value 100nF -> 2.2uF; footprint Capacitor_SMD:C_0805_2012Metric_Pad1.18x1.45mm_HandSolder -> Capacitor_SMD:C_0603_1608Metric_Pad1.08x0.95mm_HandSolder
- C3: value 100nF -> 2.2nf; footprint Capacitor_SMD:C_0805_2012Metric_Pad1.18x1.45mm_HandSolder -> Capacitor_SMD:C_0603_1608Metric_Pad1.08x0.95mm_HandSolder
- C4: value 0.1uf -> 1uf; footprint Capacitor_SMD:C_0805_2012Metric_Pad1.18x1.45mm_HandSolder -> Capacitor_SMD:C_0603_1608Metric_Pad1.08x0.95mm_HandSolder
- C5: value 2.2uF -> 56pF; footprint Capacitor_SMD:C_0402_1005Metric_Pad0.74x0.62mm_HandSolder -> Capacitor_SMD:C_0603_1608Metric_Pad1.08x0.95mm_HandSolder
- C6: value 2.2nf -> 2200pf
- C7: value 56pF -> 10nf; footprint Capacitor_SMD:C_0402_1005Metric_Pad0.74x0.62mm_HandSolder -> Capacitor_SMD:C_0603_1608Metric_Pad1.08x0.95mm_HandSolder
- C8: value 1uf -> 22UF; footprint Capacitor_SMD:C_0805_2012Metric_Pad1.18x1.45mm_HandSolder -> Capacitor_SMD:C_1206_3216Metric_Pad1.33x1.80mm_HandSolder
- C9: value 2200pf -> 2.2uf; footprint Capacitor_SMD:C_0805_2012Metric_Pad1.18x1.45mm_HandSolder -> Capacitor_SMD:C_0603_1608Metric_Pad1.08x0.95mm_HandSolder
- IC1: value CM BLE -> LM5164QDDATQ1; footprint Library:CM BLE -> LIB_LM5164QDDATQ1.kicad_mod files:SOIC127P600X170-9N
- IC2: value LM5164QDDATQ1 -> CM BLE; footprint LIB_LM5164QDDATQ1.kicad_mod files:SOIC127P600X170-9N -> Library:CM BLE
- L1: footprint Inductor_SMD:L_0402_1005Metric_Pad0.77x0.64mm_HandSolder -> Library:INR33
- L2: footprint Inductor_SMD:L_0805_2012Metric_Pad1.15x1.40mm_HandSolder -> LIB_1267AY-101M=P3.kicad_mod files:1267AY6R8NP3
- R10: value 100k -> 180k ohm
- R11: value 100E -> 20k ohm
- R12: value 100E -> 10k
- R13: value 100k -> 100R
- R14: value 100k -> 10k
- R15, R16: value 100E -> 0R
- R18: value 120R -> 0R
- R19, R26: value 0R -> 100k
- R2: value 1k -> 56k
- R21: value 10k -> 100E
- R22: value 56k -> 100E
- R22: value 1M1 -> 100E
- R23: value 120R -> 100E
- R23: value 332K -> 100E
- R24: value 3M -> 100E
- R24: value 100K -> 100E
- R25: value 100E -> 100k
- R27: value 698k ohm -> 0R
- R28: value 180k ohm -> 120R
- R29: value 20k ohm -> 0R
- R3: value 100R -> 1M
- R4: value 10k -> 300K
- R6: value 0R -> 100K
- R9: value 100k -> 700k ohm
- U1: value STM32G0B1CBTx -> TPS563200; footprint Package_QFP:LQFP-48_7x7mm_P0.5mm -> Package_TO_SOT_SMD:SOT-23-6
- U2: value MAX485E -> LP2985-3.3; footprint MAX485ESA_T.kicad_mod files:SOIC127P600X175-8N -> Package_TO_SOT_SMD:SOT-23-5
- U3: value TJA1051T-3 -> STM32G0B1CBTx; footprint Package_SO:SOIC-8_3.9x4.9mm_P1.27mm -> Package_QFP:LQFP-48_7x7mm_P0.5mm
- U4: value TPS563200 -> MAX485E; footprint Package_TO_SOT_SMD:SOT-23-6 -> MAX485ESA_T.kicad_mod files:SOIC127P600X175-8N
- U5: value LP2985-3.3 -> TJA1051T-3; footprint Package_TO_SOT_SMD:SOT-23-5 -> Package_SO:SOIC-8_3.9x4.9mm_P1.27mm
- moved L1 8.03 mm to (140.9, 52.8)
Connections:
- C1 pad 1: /3V3 -> VBST
- C1 pad 2: GND -> SW2
- C10 pad 1: /12V -> /POWER_UNIT/12Vcc
- C11 pad 1: /12V -> /STM32MCU/3V3
- C12 pad 1: Net-(U5-BP) -> /STM32MCU/3V3
- C13 pad 1: /3V3 -> /STM32MCU/3V3
- C2 pad 1: /3V3 -> Net-(IC1-GND)
- C2 pad 2: GND -> 100V
- C3 pad 1: /3V3 -> Net-(IC1-SW)
- C3 pad 2: GND -> Net-(IC1-BST)
- C4 pad 1: VBST -> 5V
- C4 pad 2: SW2 -> GND
- C5 pad 1: Net-(IC2-GND) -> Net-(IC1-FB)
- C5 pad 2: 100V -> Net-(C5-Pad2)
- C6 pad 1: Net-(IC2-SW) -> Net-(C5-Pad2)
- C6 pad 2: Net-(IC2-BST) -> /POWER_UNIT/12Vcc
- C7 pad 1: Net-(IC2-FB) -> Net-(U2-BP)
- C7 pad 2: Net-(C7-Pad2) -> GND
- C8 pad 1: 5V -> /POWER_UNIT/12Vcc
- C9 pad 1: Net-(C7-Pad2) -> /POWER_UNIT/3V3
- C9 pad 2: /12V -> GND
- E1 pad 1: /3V3 -> /STM32MCU/3V3
- E1 pad 2: /3V3 -> /STM32MCU/3V3
- IC1 pad 1: SWDIO -> Net-(IC1-GND)
- IC1 pad 2: SWCLK -> 100V
- IC1 pad 3: /RST -> Net-(IC1-EN/UVLO)
- IC1 pad 4: unconnected-(IC1-P20-Pad4) -> Net-(IC1-RON)
- IC1 pad 5: unconnected-(IC1-P18-Pad5) -> Net-(IC1-FB)
- IC1 pad 7: unconnected-(IC1-P15-Pad7) -> Net-(IC1-BST)
- IC1 pad 8: unconnected-(IC1-P14-Pad8) -> Net-(IC1-SW)
- IC1 pad 9: /TX -> GND
- IC2 pad 1: Net-(IC2-GND) -> SWDIO
- IC2 pad 2: 100V -> SWCLK
- IC2 pad 3: Net-(IC2-EN/UVLO) -> /Ble Unit/RST
- IC2 pad 4: Net-(IC2-RON) -> unconnected-(IC2-P20-Pad4)
- IC2 pad 5: Net-(IC2-FB) -> unconnected-(IC2-P18-Pad5)
- IC2 pad 7: Net-(IC2-BST) -> unconnected-(IC2-P15-Pad7)
- IC2 pad 8: Net-(IC2-SW) -> unconnected-(IC2-P14-Pad8)
- IC2 pad 9: unconnected-(IC2-EP-Pad9) -> /Ble Unit/TX
- L1 pad 2: 5V -> 5Vcc
- L2 pad 1: Net-(IC2-SW) -> Net-(IC1-SW)
- L2 pad 2: /12V -> /POWER_UNIT/12Vcc
- R1 pad 1: /3V3 -> GND
- R1 pad 2: /NRST -> VFB
- R10 pad 1: /3V3 -> /POWER_UNIT/12Vcc
- R10 pad 2: SDA_PB7 -> Net-(IC1-FB)
- R11 pad 1: SCK_2 -> Net-(IC1-FB)
- R11 pad 2: SCL_PB4 -> GND
- R12 pad 1: SDA_2 -> /STM32MCU/3V3
- R12 pad 2: SDA_PB7 -> /STM32MCU/NRST
- R13 pad 1: /3V3 -> Net-(U3-PA0)
- R13 pad 2: SCL_PB3 -> PA3
- R14 pad 1: /3V3 -> SWCLK
- R14 pad 2: SDA_PB4 -> GND
- R15 pad 1: SCK -> 5V
- R15 pad 2: SCL_PB6 -> Net-(J2-Pin_1)
- R16 pad 1: SDA1 -> /STM32MCU/12V
- R16 pad 2: SDA_PB7 -> Net-(J2-Pin_1)
- R17 pad 1: SDA_PB7 -> SCK
- R17 pad 2: Net-(J2-Pin_3) -> Net-(J2-Pin_2)
- R18 pad 1: Net-(J5-Pin_2) -> Net-(J2-Pin_2)
- R18 pad 2: Net-(J5-Pin_1) -> L
- R19 pad 1: Net-(J2-Pin_3) -> /STM32MCU/3V3
- R19 pad 2: H -> SCL_PB6
- R2 pad 1: /RX -> VFB
- R2 pad 2: /TX -> 5Vcc
- R20 pad 1: Net-(U3-S) -> /STM32MCU/3V3
- R20 pad 2: GND -> SDA_PB7
- R21 pad 1: GND -> SCK
- R21 pad 2: VFB -> SCL_PB6
- R22 pad 1: VFB -> SDA1
- R22 pad 2: 5V -> SDA_PB7
- R22 pad 1: 100V -> SDA1
- R22 pad 2: Net-(IC2-EN/UVLO) -> SDA_PB7
- R23 pad 1: L -> SCK_2
- R23 pad 2: H -> SCL_PB3
- R23 pad 1: Net-(IC2-EN/UVLO) -> SCK_2
- R23 pad 2: GND -> SCL_PB3
- R24 pad 1: Net-(D1-K) -> SDA_2
- R24 pad 2: GND -> SDA_PB4 (x2)
- R24 pad 1: Net-(IC2-RON) -> SDA_2
- R25 pad 1: PA3 -> /STM32MCU/3V3
- R25 pad 2: Net-(D1-K) -> SCL_PB3
- R26 pad 1: 5V -> /STM32MCU/3V3
- R26 pad 2: Net-(BZ1--) -> SDA_PB4
- R27 pad 1: Net-(IC2-SW) -> SDA_PB7
- R27 pad 2: Net-(C7-Pad2) -> Net-(J2-Pin_3)
- R28 pad 1: /12V -> Net-(J5-Pin_2)
- R28 pad 2: Net-(IC2-FB) -> Net-(J5-Pin_1)
- R29 pad 1: Net-(IC2-FB) -> Net-(J2-Pin_3)
- R29 pad 2: GND -> H
- R3 pad 1: Net-(U1-PA0) -> 100V
- R3 pad 2: PA3 -> Net-(IC1-EN/UVLO)
- R4 pad 1: SWCLK -> Net-(IC1-EN/UVLO)
- R5 pad 1: 5V -> /POWER_UNIT/12Vcc
- R5 pad 2: Net-(J2-Pin_1) -> /POWER_UNIT/12V
- R6 pad 1: /12V -> Net-(IC1-RON)
- R6 pad 2: Net-(J2-Pin_1) -> GND
- R7 pad 1: SCK -> /POWER_UNIT/12Vcc
- R7 pad 2: Net-(J2-Pin_2) -> /POWER_UNIT/12V
- R8 pad 1: Net-(J2-Pin_2) -> 5Vcc
- R8 pad 2: L -> 5V
- R9 pad 1: /3V3 -> Net-(IC1-SW)
- R9 pad 2: SCL_PB6 -> Net-(C5-Pad2)
- U1 pad 1: unconnected-(U1-PC13-Pad1) -> GND
- U1 pad 2: unconnected-(U1-PC14-Pad2) -> SW2
- U1 pad 3: unconnected-(U1-PC15-Pad3) -> /POWER_UNIT/12V
- U1 pad 4: /3V3 -> VFB
- U1 pad 5: /3V3 -> /POWER_UNIT/12V
- U1 pad 6: /3V3 -> VBST
- U2 pad 1: /RX -> 5V
- U2 pad 2: unconnected-(U2-~{RE}-Pad2) -> GND
- U2 pad 3: unconnected-(U2-DE-Pad3) -> 5V
- U2 pad 4: /TX -> Net-(U2-BP)
- U2 pad 5: GND -> /POWER_UNIT/3V3
- U3 pad 1: /TX -> unconnected-(U3-PC13-Pad1)
- U3 pad 2: GND -> unconnected-(U3-PC14-Pad2)
- U3 pad 3: 5V -> unconnected-(U3-PC15-Pad3)
- U3 pad 4: /RX -> /STM32MCU/3V3
- U3 pad 5: /3V3 -> /STM32MCU/3V3
- U3 pad 6: L -> /STM32MCU/3V3
- U3 pad 7: H -> GND
- U3 pad 8: Net-(U3-S) -> unconnected-(U3-PF0-Pad8)
- U4 pad 1: GND -> /STM32MCU/RX
- U4 pad 2: SW2 -> unconnected-(U4-~{RE}-Pad2)
- U4 pad 3: /12V -> unconnected-(U4-DE-Pad3)
- U4 pad 4: VFB -> /STM32MCU/TX
- U4 pad 5: /12V -> GND
- U4 pad 6: VBST -> Net-(J5-Pin_2)
- U5 pad 1: 5V -> /Tranceiver/TX
- U5 pad 4: Net-(U5-BP) -> /Tranceiver/RX
- U5 pad 5: /3V3 -> /Tranceiver/3V3

Commit message: pcb
Parts:
- moved R6 82.3 mm to (49.8, 48.5), turned to 0 degrees
- moved C9 75.6 mm to (54.4, 57.0), turned to -90 degrees
- moved C4 73.4 mm to (56.9, 58.2), turned to 180 degrees
- moved L1 73.3 mm to (67.6, 54.9)
- moved C7 71.3 mm to (54.4, 53.7), turned to 90 degrees
- moved U2 70.4 mm to (57.3, 55.6), turned to 180 degrees
- moved F1 68.6 mm to (45.7, 45.2)
- moved C6 67.9 mm to (57.1, 49.5), turned to 0 degrees
- moved C2 66.1 mm to (46.5, 42.7), turned to 180 degrees
- moved L2 66.1 mm to (63.2, 46.5), turned to -90 degrees
- moved R3 61.8 mm to (47.2, 45.2), turned to -90 degrees
- moved C10 61.5 mm to (68.8, 49.5), turned to -90 degrees
- moved C8 59.0 mm to (68.8, 44.4), turned to 90 degrees
- moved C5 58.6 mm to (56.4, 47.0), turned to -90 degrees
- moved IC1 58.1 mm to (51.9, 44.8), turned to 0 degrees
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
Commit message: buck
Connections:
- C11 pad 1: /STM32MCU/3V3 -> 3V3
- C12 pad 1: /STM32MCU/3V3 -> 3V3
- C13 pad 1: /STM32MCU/3V3 -> 3V3
- C17 pad 1: /Ina_228/3V3 -> 3V3
- C9 pad 1: /POWER_UNIT/3V3 -> 3V3
- E1 pad 1: /STM32MCU/3V3 -> 3V3
- E1 pad 2: /STM32MCU/3V3 -> 3V3
- IC2 pad 18: /Ble Unit/3V3 -> 3V3
- IC2 pad 19: /Ble Unit/3V3 -> 3V3
- IC2 pad 20: /Ble Unit/3V3 -> 3V3
- R12 pad 1: /STM32MCU/3V3 -> 3V3
- R19 pad 1: /STM32MCU/3V3 -> 3V3
- R20 pad 1: /STM32MCU/3V3 -> 3V3
- R25 pad 1: /STM32MCU/3V3 -> 3V3
- R26 pad 1: /STM32MCU/3V3 -> 3V3
- R40 pad 1: /Ina_228/3V3 -> 3V3
- R41 pad 1: /Ina_228/3V3 -> 3V3
- R42 pad 1: /Ina_228/3V3 -> 3V3
- U2 pad 5: /POWER_UNIT/3V3 -> 3V3
- U3 pad 4: /STM32MCU/3V3 -> 3V3
- U3 pad 5: /STM32MCU/3V3 -> 3V3
- U3 pad 6: /STM32MCU/3V3 -> 3V3
- U5 pad 5: /Tranceiver/3V3 -> 3V3
- U6 pad 6: /Ina_228/3V3 -> 3V3

Commit message: new
Parts:
- removed the R22 at (126.5, 55.4)
- removed the R23 at (112.3, 56.7)
- removed the R24 at (114.8, 59.9)
- moved R40 172.6 mm to (53.1, 62.6), turned to 90 degrees
- moved R34 148.2 mm to (54.6, 64.2), turned to -90 degrees
- moved R33 145.7 mm to (57.3, 65.8)
- moved R21 78.5 mm to (48.5, 62.6), turned to 90 degrees
- moved R27 78.3 mm to (50.0, 62.6)
- moved C11 77.6 mm to (52.8, 54.0), turned to 90 degrees
- moved R24 75.5 mm to (43.9, 62.6), turned to 90 degrees
- moved R23 75.2 mm to (40.9, 62.6), turned to 90 degrees
- moved R26 73.8 mm to (45.5, 62.6), turned to 90 degrees
- moved R29 73.2 mm to (54.6, 67.5), turned to 90 degrees
- moved R18 73.0 mm to (54.6, 60.8), turned to -90 degrees
- moved R25 71.5 mm to (42.4, 62.6), turned to 90 degrees
- moved C13 69.8 mm to (52.8, 57.4), turned to -90 degrees
- moved C12 67.9 mm to (54.4, 54.3), turned to 90 degrees
- moved IC2 66.8 mm to (46.6, 72.6), turned to 180 degrees
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Other:
- board size 47.2 x 46.7 mm -> 40.1 x 40.9 mm

Commit message: SOC
Parts:
- moved R30 151.2 mm to (55.0, 80.3)
- moved R31 151.0 mm to (55.0, 81.8), turned to 180 degrees
- moved R32 135.3 mm to (68.2, 67.3)
- moved H6 117.5 mm to (51.1, 35.8)
- moved J3 95.8 mm to (34.3, 60.2), turned to -90 degrees
- moved H5 95.2 mm to (72.1, 62.2)
- moved U4 84.5 mm to (65.9, 61.3), turned to -90 degrees
- moved R17 69.8 mm to (39.4, 63.1)
- moved Q1 64.5 mm to (56.6, 73.6), turned to 90 degrees
- moved R28 63.2 mm to (64.9, 65.8), turned to 0 degrees
- moved R14 63.2 mm to (39.6, 58.4)
- moved J2 61.3 mm to (45.9, 39.8)
- moved D1 60.7 mm to (54.9, 78.7), turned to 0 degrees
- moved R5 60.2 mm to (65.6, 51.6), turned to 180 degrees
- moved H3 58.4 mm to (32.8, 80.8)
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Other:
- board size 40.1 x 40.9 mm -> 44.7 x 50.3 mm

Commit message: New
Parts:
- removed BZ1: Buzzer, Buzzer_Beeper:Indicator_PUI_AI-1440-TWT-24V-2-R
- removed C1: 0.1uf, Capacitor_SMD:C_0603_1608Metric_Pad1.08x0.95mm_HandSolder
- removed C10, C8: 22UF, Capacitor_SMD:C_1206_3216Metric_Pad1.33x1.80mm_HandSolder
- removed C11: 1uF, Capacitor_SMD:C_0603_1608Metric_Pad1.08x0.95mm_HandSolder
- removed C12, C13: 100nF, Capacitor_SMD:C_0603_1608Metric_Pad1.08x0.95mm_HandSolder
- removed C14, C15, C16, C17: 22uF, Capacitor_SMD:C_1206_3216Metric_Pad1.33x1.80mm_HandSolder
- removed C2: 2.2uF, Capacitor_SMD:C_0603_1608Metric_Pad1.08x0.95mm_HandSolder
- removed C3: 2.2nf, Capacitor_SMD:C_0603_1608Metric_Pad1.08x0.95mm_HandSolder
- removed C4: 1uf, Capacitor_SMD:C_0603_1608Metric_Pad1.08x0.95mm_HandSolder
- removed C5: 56pF, Capacitor_SMD:C_0603_1608Metric_Pad1.08x0.95mm_HandSolder
- removed C6: 2200pf, Capacitor_SMD:C_0603_1608Metric_Pad1.08x0.95mm_HandSolder
- removed C7: 10nf, Capacitor_SMD:C_0603_1608Metric_Pad1.08x0.95mm_HandSolder
- removed C9: 2.2uf, Capacitor_SMD:C_0603_1608Metric_Pad1.08x0.95mm_HandSolder
- removed D1: 5.6V, Diode_SMD:D_0603_1608Metric_Pad1.05x0.95mm_HandSolder
- removed E1: LI0603G121R-10, LI0603G121R-10.kicad_mod files:FB_LI0603G121R-10
- removed F1: Fuse, Fuse:Fuse_0603_1608Metric_Pad1.05x0.95mm_HandSolder
- removed IC1: LM5164QDDATQ1, LIB_LM5164QDDATQ1.kicad_mod files:SOIC127P600X170-9N
- removed IC2: CM BLE, Library:CM BLE
- removed J1: PRG, TerminalBlock:TerminalBlock_bornier-3_P5.08mm
- removed J2: Conn_01x05_Socket, Connector_JST:JST_PH_S5B-PH-K_1x05_P2.00mm_Horizontal
- removed J3, J4: OLED, TerminalBlock:TerminalBlock_bornier-4_P5.08mm
- removed J5: Conn_01x02_Socket, TerminalBlock:TerminalBlock_bornier-2_P5.08mm
- removed J6, J7: Conn_01x02_Pin, TerminalBlock:TerminalBlock_bornier-2_P5.08mm
- removed L1: 3.3uH, Library:INR33
- removed L2: 100uH, LIB_1267AY-101M=P3.kicad_mod files:1267AY6R8NP3
- removed Q1: NDT3055L, Package_TO_SOT_SMD:SOT-223-3_TabPin2
- removed R1, R12, R14, R35, R36, R40, R41, R42: 10k, Resistor_SMD:R_0603_1608Metric_Pad0.98x0.95mm_HandSolder
- removed R10: 180k ohm, Resistor_SMD:R_0603_1608Metric_Pad0.98x0.95mm_HandSolder
- removed R11: 20k ohm, Resistor_SMD:R_0603_1608Metric_Pad0.98x0.95mm_HandSolder
- removed R13, R37, R39: 100R, Resistor_SMD:R_0603_1608Metric_Pad0.98x0.95mm_HandSolder
- removed R15, R16, R17, R18, R27, R29, R32, R5, R7, R8: 0R, Resistor_SMD:R_0603_1608Metric_Pad0.98x0.95mm_HandSolder
- removed R19, R20, R25, R26, R33: 100k, Resistor_SMD:R_0603_1608Metric_Pad0.98x0.95mm_HandSolder
- removed R2: 56k, Resistor_SMD:R_0603_1608Metric_Pad0.98x0.95mm_HandSolder
- removed R21, R22, R23, R24, R31: 100E, Resistor_SMD:R_0603_1608Metric_Pad0.98x0.95mm_HandSolder
- removed R28, R34: 120R, Resistor_SMD:R_0603_1608Metric_Pad0.98x0.95mm_HandSolder
- removed R3: 1M, Resistor_SMD:R_0603_1608Metric_Pad0.98x0.95mm_HandSolder
- removed R30: 3M, Resistor_SMD:R_0603_1608Metric_Pad0.98x0.95mm_HandSolder
- removed R38: 16.2M, Resistor_SMD:R_0603_1608Metric_Pad0.98x0.95mm_HandSolder
- removed R4: 300K, Resistor_SMD:R_0603_1608Metric_Pad0.98x0.95mm_HandSolder
- removed R6: 100K, Resistor_SMD:R_0603_1608Metric_Pad0.98x0.95mm_HandSolder
- removed R9: 700k ohm, Resistor_SMD:R_0603_1608Metric_Pad0.98x0.95mm_HandSolder
- removed U1: TPS563200, Package_TO_SOT_SMD:SOT-23-6
- removed U2: LP2985-3.3, Package_TO_SOT_SMD:SOT-23-5
- removed U3: STM32G0B1CBTx, Package_QFP:LQFP-48_7x7mm_P0.5mm
- removed U4: MAX485E, MAX485ESA_T.kicad_mod files:SOIC127P600X175-8N
- removed U5: TJA1051T-3, Package_SO:SOIC-8_3.9x4.9mm_P1.27mm
- removed U6: INA228AQDGSRQ1, Package_SO:VSSOP-10_3x3mm_P0.5mm
- added BZ301: Buzzer, Buzzer_Beeper:Indicator_PUI_AI-1440-TWT-24V-2-R, F.Cu at (131.4, 29.8)
- added C101: 0.1uf, Capacitor_SMD:C_0603_1608Metric_Pad1.08x0.95mm_HandSolder, F.Cu at (89.3, 63.5)
- added C102: 2.2uF, Capacitor_SMD:C_0603_1608Metric_Pad1.08x0.95mm_HandSolder, F.Cu at (91.0, 116.1)
- added C103: 2.2nf, Capacitor_SMD:C_0603_1608Metric_Pad1.08x0.95mm_HandSolder, F.Cu at (100.2, 116.1)
- added C104: 1uf, Capacitor_SMD:C_0603_1608Metric_Pad1.08x0.95mm_HandSolder, F.Cu at (89.3, 71.1)
- added C105: 56pF, Capacitor_SMD:C_0603_1608Metric_Pad1.08x0.95mm_HandSolder, F.Cu at (99.5, 121.9)
- added C106: 2200pf, Capacitor_SMD:C_0603_1608Metric_Pad1.08x0.95mm_HandSolder, F.Cu at (107.6, 121.9)
- added C107: 10nf, Capacitor_SMD:C_0603_1608Metric_Pad1.08x0.95mm_HandSolder, F.Cu at (89.3, 78.6)
- added C108: 22UF, Capacitor_SMD:C_1206_3216Metric_Pad1.33x1.80mm_HandSolder, F.Cu at (90.1, 81.5)
- added C109: 2.2uf, Capacitor_SMD:C_0603_1608Metric_Pad1.08x0.95mm_HandSolder, F.Cu at (93.7, 63.5)
- added C110: 22UF, Capacitor_SMD:C_1206_3216Metric_Pad1.33x1.80mm_HandSolder, F.Cu at (105.3, 111.2)
- added C201: 1uF, Capacitor_SMD:C_0603_1608Metric_Pad1.08x0.95mm_HandSolder, F.Cu at (103.3, 41.4)
- added C202: 100nF, Capacitor_SMD:C_0603_1608Metric_Pad1.08x0.95mm_HandSolder, F.Cu at (103.3, 44.0)
- added C203: 100nF, Capacitor_SMD:C_0603_1608Metric_Pad1.08x0.95mm_HandSolder, F.Cu at (103.3, 46.5)
- added C601: 22uF, Capacitor_SMD:C_1206_3216Metric_Pad1.33x1.80mm_HandSolder, F.Cu at (146.4, 49.4)
- added C602: 22uF, Capacitor_SMD:C_1206_3216Metric_Pad1.33x1.80mm_HandSolder, F.Cu at (146.4, 52.7)
- added C603: 22uF, Capacitor_SMD:C_1206_3216Metric_Pad1.33x1.80mm_HandSolder, F.Cu at (146.4, 56.1)
- added C604: 22uF, Capacitor_SMD:C_1206_3216Metric_Pad1.33x1.80mm_HandSolder, F.Cu at (146.4, 59.4)
- added D301: 5.6V, Diode_SMD:D_0603_1608Metric_Pad1.05x0.95mm_HandSolder, F.Cu at (144.0, 38.7)
- added E201: LI0603G121R-10, LI0603G121R-10.kicad_mod files:FB_LI0603G121R-10, F.Cu at (111.0, 32.3)
- added F201: Fuse, Fuse:Fuse_0603_1608Metric_Pad1.05x0.95mm_HandSolder, F.Cu at (87.9, 117.9)
- added IC101: LM5164QDDATQ1, LIB_LM5164QDDATQ1.kicad_mod files:SOIC127P600X170-9N, F.Cu at (95.6, 117.3)
- added IC501: CM BLE, Library:CM BLE, F.Cu at (135.2, 81.9)
- added J201: PRG, TerminalBlock:TerminalBlock_bornier-3_P5.08mm, F.Cu at (112.1, 26.6)
- added J202: Conn_01x05_Socket, Connector_JST:JST_PH_S5B-PH-K_1x05_P2.00mm_Horizontal, F.Cu at (90.1, 42.6)
- added J203: OLED, TerminalBlock:TerminalBlock_bornier-4_P5.08mm, F.Cu at (90.4, 26.6)
- added J204: OLED, TerminalBlock:TerminalBlock_bornier-4_P5.08mm, F.Cu at (90.4, 35.7)
- added J205: Conn_01x02_Socket, TerminalBlock:TerminalBlock_bornier-2_P5.08mm, F.Cu at (90.4, 54.4)
- added J601: Conn_01x02_Pin, TerminalBlock:TerminalBlock_bornier-2_P5.08mm, F.Cu at (135.1, 52.2)
- added J602: Conn_01x02_Pin, TerminalBlock:TerminalBlock_bornier-2_P5.08mm, F.Cu at (135.1, 61.3)
- added L101: 3.3uH, Library:INR33, F.Cu at (96.2, 82.6)
- added L102: 100uH, LIB_1267AY-101M=P3.kicad_mod files:1267AY6R8NP3, F.Cu at (105.5, 116.8)
- added Q301: NDT3055L, Package_TO_SOT_SMD:SOT-223-3_TabPin2, F.Cu at (132.5, 41.6)
- added R101: 10k, Resistor_SMD:R_0603_1608Metric_Pad0.98x0.95mm_HandSolder, F.Cu at (93.7, 66.0)
- added R102: 56k, Resistor_SMD:R_0603_1608Metric_Pad0.98x0.95mm_HandSolder, F.Cu at (82.6, 76.5)
- added R103: 1M, Resistor_SMD:R_0603_1608Metric_Pad0.98x0.95mm_HandSolder, F.Cu at (89.4, 117.9)
- added R104: 300K, Resistor_SMD:R_0603_1608Metric_Pad0.98x0.95mm_HandSolder, F.Cu at (91.0, 119.5)
- added R105: 0R, Resistor_SMD:R_0603_1608Metric_Pad0.98x0.95mm_HandSolder, F.Cu at (50.7, 106.1)
- added R106: 100K, Resistor_SMD:R_0603_1608Metric_Pad0.98x0.95mm_HandSolder, F.Cu at (92.7, 121.9)
- added R107: 0R, Resistor_SMD:R_0603_1608Metric_Pad0.98x0.95mm_HandSolder, F.Cu at (98.0, 63.5)
- added R108: 0R, Resistor_SMD:R_0603_1608Metric_Pad0.98x0.95mm_HandSolder, F.Cu at (98.0, 66.0)
- added R109: 700k ohm, Resistor_SMD:R_0603_1608Metric_Pad0.98x0.95mm_HandSolder, F.Cu at (103.6, 121.9)
- added R110: 180k ohm, Resistor_SMD:R_0603_1608Metric_Pad0.98x0.95mm_HandSolder, F.Cu at (99.5, 123.4)
- added R111: 20k ohm, Resistor_SMD:R_0603_1608Metric_Pad0.98x0.95mm_HandSolder, F.Cu at (96.0, 121.9)
- added R201: 10k, Resistor_SMD:R_0603_1608Metric_Pad0.98x0.95mm_HandSolder, F.Cu at (103.3, 51.5)
- added R202: 100R, Resistor_SMD:R_0603_1608Metric_Pad0.98x0.95mm_HandSolder, F.Cu at (103.3, 54.0)
- added R203: 10k, Resistor_SMD:R_0603_1608Metric_Pad0.98x0.95mm_HandSolder, F.Cu at (103.3, 56.5)
- added R204: 0R, Resistor_SMD:R_0603_1608Metric_Pad0.98x0.95mm_HandSolder, F.Cu at (103.3, 59.0)
- added R205: 0R, Resistor_SMD:R_0603_1608Metric_Pad0.98x0.95mm_HandSolder, F.Cu at (107.6, 41.4)
- added R206: 0R, Resistor_SMD:R_0603_1608Metric_Pad0.98x0.95mm_HandSolder, F.Cu at (107.6, 44.0)
- added R207: 0R, Resistor_SMD:R_0603_1608Metric_Pad0.98x0.95mm_HandSolder, F.Cu at (107.6, 46.5)
- added R208: 100k, Resistor_SMD:R_0603_1608Metric_Pad0.98x0.95mm_HandSolder, F.Cu at (107.6, 49.0)
- added R209: 100k, Resistor_SMD:R_0603_1608Metric_Pad0.98x0.95mm_HandSolder, F.Cu at (107.6, 51.5)
- added R210: 100E, Resistor_SMD:R_0603_1608Metric_Pad0.98x0.95mm_HandSolder, F.Cu at (107.6, 54.0)
- added R211: 100E, Resistor_SMD:R_0603_1608Metric_Pad0.98x0.95mm_HandSolder, F.Cu at (107.6, 56.5)
- added R212: 100E, Resistor_SMD:R_0603_1608Metric_Pad0.98x0.95mm_HandSolder, F.Cu at (107.6, 59.0)
- added R213: 100E, Resistor_SMD:R_0603_1608Metric_Pad0.98x0.95mm_HandSolder, F.Cu at (112.0, 41.4)
- added R214: 100k, Resistor_SMD:R_0603_1608Metric_Pad0.98x0.95mm_HandSolder, F.Cu at (112.0, 44.0)
- added R215: 100k, Resistor_SMD:R_0603_1608Metric_Pad0.98x0.95mm_HandSolder, F.Cu at (112.0, 46.5)
- added R216: 0R, Resistor_SMD:R_0603_1608Metric_Pad0.98x0.95mm_HandSolder, F.Cu at (112.0, 49.0)
- added R217: 120R, Resistor_SMD:R_0603_1608Metric_Pad0.98x0.95mm_HandSolder, F.Cu at (112.0, 51.5)
- added R218: 0R, Resistor_SMD:R_0603_1608Metric_Pad0.98x0.95mm_HandSolder, F.Cu at (112.0, 54.0)
- added R301: 3M, Resistor_SMD:R_0603_1608Metric_Pad0.98x0.95mm_HandSolder, F.Cu at (139.6, 38.7)
- added R302: 100E, Resistor_SMD:R_0603_1608Metric_Pad0.98x0.95mm_HandSolder, F.Cu at (139.6, 41.2)
- added R303: 0R, Resistor_SMD:R_0603_1608Metric_Pad0.98x0.95mm_HandSolder, F.Cu at (139.6, 43.7)
- added R401: 100k, Resistor_SMD:R_0603_1608Metric_Pad0.98x0.95mm_HandSolder, F.Cu at (146.9, 80.0)
- added R402: 120R, Resistor_SMD:R_0603_1608Metric_Pad0.98x0.95mm_HandSolder, F.Cu at (146.9, 82.6)
- added R601: 10k, Resistor_SMD:R_0603_1608Metric_Pad0.98x0.95mm_HandSolder, F.Cu at (129.7, 48.9)
- added R602: 10k, Resistor_SMD:R_0603_1608Metric_Pad0.98x0.95mm_HandSolder, F.Cu at (129.7, 51.5)
- added R603: 100R, Resistor_SMD:R_0603_1608Metric_Pad0.98x0.95mm_HandSolder, F.Cu at (129.7, 54.0)
- added R604: 16.2M, Resistor_SMD:R_0603_1608Metric_Pad0.98x0.95mm_HandSolder, F.Cu at (129.7, 56.5)
- added R605: 100R, Resistor_SMD:R_0603_1608Metric_Pad0.98x0.95mm_HandSolder, F.Cu at (129.7, 59.0)
- added R606: 10k, Resistor_SMD:R_0603_1608Metric_Pad0.98x0.95mm_HandSolder, F.Cu at (129.7, 61.5)
- added R607: 10k, Resistor_SMD:R_0603_1608Metric_Pad0.98x0.95mm_HandSolder, F.Cu at (129.7, 64.0)
- added R608: 10k, Resistor_SMD:R_0603_1608Metric_Pad0.98x0.95mm_HandSolder, F.Cu at (129.7, 66.5)
- added U101: TPS563200, Package_TO_SOT_SMD:SOT-23-6, F.Cu at (64.0, 118.9)
- added U102: LP2985-3.3, Package_TO_SOT_SMD:SOT-23-5, F.Cu at (102.8, 85.3)
- added U201: STM32G0B1CBTx, Package_QFP:LQFP-48_7x7mm_P0.5mm, F.Cu at (119.8, 45.9)
- added U202: MAX485E, MAX485ESA_T.kicad_mod files:SOIC127P600X175-8N, F.Cu at (119.3, 54.8)
- added U401: TJA1051T-3, Package_SO:SOIC-8_3.9x4.9mm_P1.27mm, F.Cu at (149.0, 75.6)
- added U601: INA228AQDGSRQ1, Package_SO:VSSOP-10_3x3mm_P0.5mm, F.Cu at (135.6, 68.1)
- moved H3 57.1 mm to (20.5, 25.0)
- moved H5 44.9 mm to (76.2, 17.5)
- moved H6 21.2 mm to (62.9, 18.3)
- moved H1 17.5 mm to (32.9, 18.1)
Routing:
- net GND: vias 0 -> 2
