File: SOC DISPLAY.kicad_sch (KiCad schematic)
At the start: 64 parts, among them IC1 CM BLE, IC2 LM5164QDDATQ1, J2 PRG, J3 OLED, U2 LP2985-3.3, U3 TPS563200, U4 STM32G0B1CBTx, U7 TJA1051T-3

Commit message: changes
Parts:
- removed FB1: FerriteBead, symbol Device:FerriteBead
- added E1: LI0603G121R-10, LI0603G121R-10.kicad_mod files:FB_LI0603G121R-10, symbol LI0603G121R-10:LI0603G121R-10
- 100k1, 1M1, 332k1: footprint (none) -> Resistor_SMD:R_0603_1608Metric_Pad0.98x0.95mm_HandSolder
Connections:
- net Vdd: now also E1.1, E1.2
Changed lines of the file:
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@@
     (stroke (width 0) (type default))
   )
-  (wire (pts (xy 48.26 22.86) (xy 48.26 24.13))
+  (wire (pts (xy 48.26 19.05) (xy 48.26 24.13))
     (stroke (width 0) (type default))
   )
@@
     (stroke (width 0) (type default))
   )
-  (wire (pts (xy 21.59 22.86) (xy 48.26 22.86))
+  (wire (pts (xy 25.4 31.75) (xy 27.94 31.75))
+    (stroke (width 0) (type default))
+  )
+  (wire (pts (xy 19.05 19.05) (xy 48.26 19.05))
     (stroke (width 0) (type default))
   )
@@
     (stroke (width 0) (type default))
   )
-  (wire (pts (xy 27.94 30.48) (xy 27.94 29.21))
+  (wire (pts (xy 25.4 34.29) (xy 25.4 31.75))
     (stroke (width 0) (type default))
   )
@@
     (stroke (width 0) (type default))
   )
-  (wire (pts (xy 21.59 30.48) (xy 27.94 30.48))
+  (wire (pts (xy 19.05 34.29) (xy 25.4 34.29))
     (stroke (width 0) (type default))
   )
@@
     (stroke (width 0) (type default))
   )
+  (wire (pts (xy 27.94 31.75) (xy 27.94 29.21))
+    (stroke (width 0) (type default))
+  )
   (wire (pts (xy 160.02 73.66) (xy 160.02 74.93))
     (stroke (width 0) (type default))
@@
     (effects (font (size 1.27 1.27)) (justify left bottom))
   )
-  (label "3V3" (at 16.51 39.37 90) (fields_autoplaced)
-    (effects (font (size 1.27 1.27)) (justify left bottom))
+  (label "3V3" (at 16.51 39.37 270) (fields_autoplaced)
+    (effects (font (size 1.27 1.27)) (justify right bottom))
   )
   (label "RX" (at 88.9 95.25 180) (fields_autoplaced)
@@
       (effects (font (size 1.27 1.27)) (justify left))
     )
-    (property "Footprint" "" (at 160.02 77.47 0)
+    (property "Footprint" "Resistor_SMD:R_0603_1608Metric_Pad0.98x0.95mm_HandSolder" (at 160.02 77.47 0)
       (effects (font (size 1.27 1.27)) hide)
     )
@@
     )
   )
+  (symbol (lib_id "LI0603G121R-10:LI0603G121R-10") (at 19.05 26.67 90) (unit 1)
+    (in_bom yes) (on_board yes) (dnp no)
+    (property "Reference" "E1" (at 20.32 24.13 90)
+      (effects (font (size 1.27 1.27)) (justify right))
+    )
+    (property "Value" "LI0603G121R-10" (at 15.24 21.59 0)
+      (effects (font (size 1.27 1.27)) (justify right))
+    )
+    (property "Footprint" "LI0603G121R-10.kicad_mod files:FB_LI0603G121R-10" (at 19.05 26.67 0)
+      (effects (font (size 1.27 1.27)) (justify left bottom) hide)
+    )
+    (property "Datasheet" "" (at 19.05 26.67 0)
+      (effects (font (size 1.27 1.27)) (justify left bottom) hide)
+    )
+    (property "PARTREV" "C" (at 19.05 26.67 0)
+      (effects (font (size 1.27 1.27)) (justify left bottom) hide)
+    )
+    (property "STANDARD" "Manufacturer Recommendations" (at 19.05 26.67 0)
+      (effects (font (size 1.27 1.27)) (justify left bottom) hide)
+    )
+    (property "MAXIMUM_PACKAGE_HEIGHT" "0.95 mm" (at 19.05 26.67 0)
+      (effects (font (size 1.27 1.27)) (justify left bottom) hide)
+    )
+    (property "MANUFACTURER" "Laird" (at 19.05 26.67 0)
+      (effects (font (size 1.27 1.27)) (justify left bottom) hide)
+    )
+    (pin "1")
+    (pin "2")
+    (instances
+      (project "SOC DISPLAY"
+        (path "/9f7696f8-e9fa-4362-b2ca-5dde3355ad01"
+          (reference "E1") (unit 1)
+        )
+      )
+    )
+  )
   (symbol (lib_id "power:GND") (at 83.82 113.03 0) (unit 1)
     (in_bom yes) (on_board yes) (dnp no) (fields_autoplaced)
@@
       (effects (font (size 1.27 1.27)) (justify left))
     )
-    (property "Footprint" "" (at 170.18 78.74 0)
+    (property "Footprint" "Resistor_SMD:R_0603_1608Metric_Pad0.98x0.95mm_HandSolder" (at 170.18 78.74 0)
       (effects (font (size 1.27 1.27)) hide)
     )
@@
     )
   )
-  (symbol (lib_id "Device:FerriteBead") (at 21.59 26.67 0) (unit 1)
-    (in_bom yes) (on_board yes) (dnp no)
-    (property "Reference" "FB1" (at 15.24 24.13 0)
-      (effects (font (size 1.27 1.27)) (justify left))
-    )
-    (property "Value" "FerriteBead" (at 17.78 33.02 90)
-      (effects (font (size 1.27 1.27)) (justify left) hide)
-    )
-    (property "Footprint" "" (at 19.812 26.67 90)
-      (effects (font (size 1.27 1.27)) hide)
-    )
-    (property "Datasheet" "~" (at 21.59 26.67 0)
-      (effects (font (size 1.27 1.27)) hide)
-    )
-    (pin "1")
-    (pin "2")
-    (instances
-      (project "SOC DISPLAY"
-        (path "/9f7696f8-e9fa-4362-b2ca-5dde3355ad01"
-          (reference "FB1") (unit 1)
-        )
-      )
-    )
-  )
   (symbol (lib_id "Mechanical:MountingHole") (at 260.35 96.52 0) (unit 1)
     (in_bom yes) (on_board yes) (dnp no)
@@
       (effects (font (size 1.27 1.27)) (justify left))
     )
-    (property "Footprint" "" (at 160.02 69.85 0)
+    (property "Footprint" "Resistor_SMD:R_0603_1608Metric_Pad0.98x0.95mm_HandSolder" (at 160.02 69.85 0)
       (effects (font (size 1.27 1.27)) hide)
     )

Commit message: 3V3
Connections:
- net Vdd renamed 3V3
Changed lines of the file:
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@@
+    (effects (font (size 1.27 1.27)) (justify right bottom))
+  )
+  (label "3V3" (at 25.4 105.41 180) (fields_autoplaced)
     (effects (font (size 1.27 1.27)) (justify right bottom))
   )
@@
     (effects (font (size 1.27 1.27)) (justify left bottom))
   )
+  (label "3V3" (at 83.82 105.41 180) (fields_autoplaced)
+    (effects (font (size 1.27 1.27)) (justify right bottom))
+  )
   (label "12V" (at 254 63.5 0) (fields_autoplaced)
     (effects (font (size 1.27 1.27)) (justify left bottom))
@@
     (effects (font (size 1.27 1.27)) (justify right bottom))
   )
+  (label "3V3" (at 78.74 105.41 180) (fields_autoplaced)
+    (effects (font (size 1.27 1.27)) (justify right bottom))
+  )
   (label "TX" (at 148.59 124.46 180) (fields_autoplaced)
     (effects (font (size 1.27 1.27)) (justify right bottom))
@@
     )
   )
-  (global_label "Vdd" (shape input) (at 78.74 105.41 90) (fields_autoplaced)
-    (effects (font (size 1.27 1.27)) (justify left))
-    (property "Intersheetrefs" "${INTERSHEET_REFS}" (at 78.74 99.1176 90)
-      (effects (font (size 1.27 1.27)) (justify left) hide)
-    )
-  )
   (global_label "SCK" (shape input) (at 102.87 30.48 180) (fields_autoplaced)
     (effects (font (size 1.27 1.27)) (justify right))
@@
     )
   )
-  (global_label "Vdd" (shape input) (at 48.26 24.13 90) (fields_autoplaced)
-    (effects (font (size 1.27 1.27)) (justify left))
-    (property "Intersheetrefs" "${INTERSHEET_REFS}" (at 48.26 17.8376 90)
-      (effects (font (size 1.27 1.27)) (justify left) hide)
-    )
-  )
   (global_label "100V" (shape input) (at 153.67 66.04 180) (fields_autoplaced)
     (effects (font (size 1.27 1.27)) (justify right))
@@
     )
   )
-  (global_label "Vref" (shape input) (at 25.4 105.41 90) (fields_autoplaced)
-    (effects (font (size 1.27 1.27)) (justify left))
-    (property "Intersheetrefs" "${INTERSHEET_REFS}" (at 25.4 98.8151 90)
-      (effects (font (size 1.27 1.27)) (justify left) hide)
-    )
-  )
   (global_label "100V" (shape input) (at 106.68 60.96 90) (fields_autoplaced)
     (effects (font (size 1.27 1.27)) (justify left))
@@
     )
   )
-  (global_label "Vref" (shape input) (at 27.94 29.21 90) (fields_autoplaced)
-    (effects (font (size 1.27 1.27)) (justify left))
-    (property "Intersheetrefs" "${INTERSHEET_REFS}" (at 27.94 22.6151 90)
-      (effects (font (size 1.27 1.27)) (justify left) hide)
-    )
-  )
   (global_label "SWCLK" (shape input) (at 26.67 142.24 180) (fields_autoplaced)
     (effects (font (size 1.27 1.27)) (justify right))
@@
     )
   )
-  (global_label "Vdd" (shape input) (at 83.82 105.41 90) (fields_autoplaced)
-    (effects (font (size 1.27 1.27)) (justify left))
-    (property "Intersheetrefs" "${INTERSHEET_REFS}" (at 83.82 99.1176 90)
-      (effects (font (size 1.27 1.27)) (justify left) hide)
-    )
-  )

Commit message: chanses made
Changed lines of the file:
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@@
-    (stroke (width 0) (type default))
-  )
-  (wire (pts (xy 25.4 31.75) (xy 27.94 31.75))
     (stroke (width 0) (type default))
   )
@@
     (stroke (width 0) (type default))
   )
+  (wire (pts (xy 27.94 30.48) (xy 27.94 29.21))
+    (stroke (width 0) (type default))
+  )
   (wire (pts (xy 88.9 95.25) (xy 93.98 95.25))
     (stroke (width 0) (type default))
@@
     (stroke (width 0) (type default))
   )
-  (wire (pts (xy 25.4 34.29) (xy 25.4 31.75))
-    (stroke (width 0) (type default))
-  )
   (wire (pts (xy 88.9 44.45) (xy 92.71 44.45))
     (stroke (width 0) (type default))
@@
     (stroke (width 0) (type default))
   )
+  (wire (pts (xy 25.4 30.48) (xy 27.94 30.48))
+    (stroke (width 0) (type default))
+  )
   (wire (pts (xy 149.86 127) (xy 151.13 127))
     (stroke (width 0) (type default))
@@
     (stroke (width 0) (type default))
   )
-  (wire (pts (xy 27.94 31.75) (xy 27.94 29.21))
-    (stroke (width 0) (type default))
-  )
+  (wire (pts (xy 25.4 34.29) (xy 25.4 30.48))
+    (stroke (width 0) (type default))
+  )

Commit message: Sch Changes
Parts:
- removed C1: 1uF, Capacitor_SMD:C_0805_2012Metric_Pad1.18x1.45mm_HandSolder, symbol Device:C
- removed C1 (x2): 100nF, Capacitor_SMD:C_0805_2012Metric_Pad1.18x1.45mm_HandSolder, symbol Device:C
- removed E1: LI0603G121R-10, LI0603G121R-10.kicad_mod files:FB_LI0603G121R-10, symbol LI0603G121R-10:LI0603G121R-10
- removed F?: Fuse, Fuse:Fuse_0603_1608Metric_Pad1.05x0.95mm_HandSolder, symbol Device:Fuse
- removed J3: OLED, TerminalBlock:TerminalBlock_bornier-4_P5.08mm, symbol Connector:Conn_01x04_Socket
- removed J?: Conn_01x02_Socket, TerminalBlock:TerminalBlock_bornier-2_P5.08mm, symbol Connector:Conn_01x02_Socket
- removed J?: Conn_01x05_Socket, Connector_JST:JST_PH_S5B-PH-K_1x05_P2.00mm_Horizontal, symbol Connector:Conn_01x05_Socket
- removed R18, R19: 100E, Resistor_SMD:R_0603_1608Metric_Pad0.98x0.95mm_HandSolder, symbol Device:R
- removed R20, R21: 100k, Resistor_SMD:R_0603_1608Metric_Pad0.98x0.95mm_HandSolder, symbol Device:R
- removed R? (x5): 0R, Resistor_SMD:R_0603_1608Metric_Pad0.98x0.95mm_HandSolder, symbol Device:R
- removed U?: MAX485E, MAX485ESA_T.kicad_mod files:SOIC127P600X175-8N, symbol Interface_UART:MAX485E
- added C1 (x2): 100nF, Capacitor_SMD:C_0805_2012Metric_Pad1.18x1.45mm_HandSolder, symbol Device:C
- added C1: 1uF, Capacitor_SMD:C_0805_2012Metric_Pad1.18x1.45mm_HandSolder, symbol Device:C
- added E?: LI0603G121R-10, LI0603G121R-10.kicad_mod files:FB_LI0603G121R-10, symbol LI0603G121R-10:LI0603G121R-10
- added F?: Fuse, Fuse:Fuse_0603_1608Metric_Pad1.05x0.95mm_HandSolder, symbol Device:Fuse
- added J3 (x2): OLED, TerminalBlock:TerminalBlock_bornier-4_P5.08mm, symbol Connector:Conn_01x04_Socket
- added J?: Conn_01x05_Socket, Connector_JST:JST_PH_S5B-PH-K_1x05_P2.00mm_Horizontal, symbol Connector:Conn_01x05_Socket
- added J?: Conn_01x02_Socket, TerminalBlock:TerminalBlock_bornier-2_P5.08mm, symbol Connector:Conn_01x02_Socket
- added R18 (x2), R19 (x2): 100E, Resistor_SMD:R_0603_1608Metric_Pad0.98x0.95mm_HandSolder, symbol Device:R
- added R20 (x2), R21 (x2): 100k, Resistor_SMD:R_0603_1608Metric_Pad0.98x0.95mm_HandSolder, symbol Device:R
- added R? (x6): 0R, Resistor_SMD:R_0603_1608Metric_Pad0.98x0.95mm_HandSolder, symbol Device:R
- added U?: MAX485E, MAX485ESA_T.kicad_mod files:SOIC127P600X175-8N, symbol Interface_UART:MAX485E
Connections:
- net 100V: now also F?.2
- net 12V: now also R?.1
- net 3V3: now also C1.1, C1.1, C1.1, E?.1, E?.2, R20.1, R20.1, R21.1, R21.1
- net 5V: now also J3.1 (Pin_1), J3.1 (Pin_1), R?.1, U?.8 (VCC)
- net GND: now also C1.2, C1.2, C1.2, J3.4 (Pin_4), J3.4 (Pin_4), J?.4 (Pin_4), U?.5 (GND)
- net H: now also R?.2
- net L: now also R?.2
- net PA3: now also J?.5 (Pin_5)
- net RX: now also U?.1 (RO)
- net SCK: now also J3.3 (Pin_3), R18.1, R?.1
- net SDA1: now also J3.2 (Pin_2), R19.1
- net TX: now also U?.4 (DI)
- net at R25.2: now also J?.1 (Pin_1), U?.7 (B)
- net at R25.1: now also J?.2 (Pin_2), U?.6 (A)
- net  SCL_PB3: now reaches U4.42 (PB3)
- net SDA_PB4: now reaches U4.43 (PB4)
- net SDA_PB4: now also R21.2
- net SCL renamed SCL_PB6
- net SCL_PB6: now also R18.2, R20.2
- net SDA renamed SDA_PB7
- net SDA_PB7: now also R19.2, R19.2, R21.2, R?.1
- new net: J?.2 (Pin_2), R?.1, R?.2
- new net: F?.1, J?.1 (Pin_1), R?.2, R?.2
- new net: J?.3 (Pin_3), R?.1, R?.2
- new net SCK_2: J3.3 (Pin_3), R18.1
- new net SCL_PB3: R20.2
- new net SCL_PB4: R18.2
- new net SDA_2: J3.2 (Pin_2), R19.1
- no-connect marks 53 -> 51

Commit message: frst
Parts:
- gave numbers to parts that had none: 1

Commit message: Matic
Connections:
- net SCL_PB4 is gone; now on net SCL_PB3: R18.2
- net SDA_PB4: now also R19.2
- net SDA_PB7: no longer R19.2
Other:
- moved on the sheet: J3, R18, R19, R20, R21

Commit message: now
Connections:
- net  SCL_PB3 is gone; now on net SCL_PB3: U4.42 (PB3)
Changed lines of the file:
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@@
     )
   )
-  (global_label " SCL_PB3" (shape input) (at 66.04 80.01 0) (fields_autoplaced)
+  (global_label "SCL_PB3" (shape input) (at 66.04 80.01 0) (fields_autoplaced)
     (effects (font (size 1.27 1.27)) (justify left))
-    (property "Intersheetrefs" "${INTERSHEET_REFS}" (at 78.1381 80.01 0)
+    (property "Intersheetrefs" "${INTERSHEET_REFS}" (at 77.1705 80.01 0)
       (effects (font (size 1.27 1.27)) (justify left) hide)
     )

Commit message: Done
Parts:
- removed 100k1: R24, Resistor_SMD:R_0603_1608Metric_Pad0.98x0.95mm_HandSolder, symbol Device:R_Small_US
- removed 1M1: R22, Resistor_SMD:R_0603_1608Metric_Pad0.98x0.95mm_HandSolder, symbol Device:R_Small_US
- removed 332k1: R23, Resistor_SMD:R_0603_1608Metric_Pad0.98x0.95mm_HandSolder, symbol Device:R_Small_US
- removed BZ?: Buzzer, Buzzer_Beeper:Indicator_PUI_AI-1440-TWT-24V-2-R, symbol Device:Buzzer
- removed C1 (x2): 100nF, Capacitor_SMD:C_0805_2012Metric_Pad1.18x1.45mm_HandSolder, symbol Device:C
- removed C1: 1uf, Capacitor_SMD:C_0805_2012Metric_Pad1.18x1.45mm_HandSolder, symbol Device:C
- removed C1: 1uF, Capacitor_SMD:C_0805_2012Metric_Pad1.18x1.45mm_HandSolder, symbol Device:C
- removed C1: 2.2uf, Capacitor_SMD:C_0805_2012Metric_Pad1.18x1.45mm_HandSolder, symbol Device:C
- removed C1: 10nf, Capacitor_SMD:C_0805_2012Metric_Pad1.18x1.45mm_HandSolder, symbol Device:C
- removed C2: 0.1uf, Capacitor_SMD:C_0805_2012Metric_Pad1.18x1.45mm_HandSolder, symbol Device:C
- removed C2: 2.2nf, Capacitor_SMD:C_0603_1608Metric_Pad1.08x0.95mm_HandSolder, symbol Device:C
- removed C3 (x2): 22UF, Capacitor_SMD:C_1206_3216Metric_Pad1.33x1.80mm_HandSolder, symbol Device:C
- removed C4: 2200pf, Capacitor_SMD:C_0805_2012Metric_Pad1.18x1.45mm_HandSolder, symbol Device:C
- removed C5: 2.2uF, Capacitor_SMD:C_0402_1005Metric_Pad0.74x0.62mm_HandSolder, symbol Device:C
- removed C5: 56pF, Capacitor_SMD:C_0402_1005Metric_Pad0.74x0.62mm_HandSolder, symbol Device:C
- removed D?: 5.6V, Diode_SMD:D_0603_1608Metric_Pad1.05x0.95mm_HandSolder, symbol Device:D_Schottky
- removed E1: LI0603G121R-10, LI0603G121R-10.kicad_mod files:FB_LI0603G121R-10, symbol LI0603G121R-10:LI0603G121R-10
- removed F?: Fuse, Fuse:Fuse_0603_1608Metric_Pad1.05x0.95mm_HandSolder, symbol Device:Fuse
- removed IC1: CM BLE, Library:CM BLE, symbol Library:COMMON_BLUETOOTH
- removed IC2: LM5164QDDATQ1, LIB_LM5164QDDATQ1.kicad_mod files:SOIC127P600X170-9N, symbol LM5164QDDATQ1:LM5164QDDATQ1
- removed J2: PRG, TerminalBlock:TerminalBlock_bornier-3_P5.08mm, symbol Connector:Conn_01x03_Socket
- removed J3 (x2): OLED, TerminalBlock:TerminalBlock_bornier-4_P5.08mm, symbol Connector:Conn_01x04_Socket
- removed J?: Conn_01x05_Socket, Connector_JST:JST_PH_S5B-PH-K_1x05_P2.00mm_Horizontal, symbol Connector:Conn_01x05_Socket
- removed J?: Conn_01x02_Socket, TerminalBlock:TerminalBlock_bornier-2_P5.08mm, symbol Connector:Conn_01x02_Socket
- removed L1: 100uH, Inductor_SMD:L_0805_2012Metric_Pad1.15x1.40mm_HandSolder, symbol Device:L
- removed L1: 3.3uH, Inductor_SMD:L_0402_1005Metric_Pad0.77x0.64mm_HandSolder, symbol Device:L
- removed Q?: NDT3055L, Package_TO_SOT_SMD:SOT-223-3_TabPin2, symbol Transistor_FET:NDT3055L
- removed R1, R6, R9: 10k, Resistor_SMD:R_0603_1608Metric_Pad0.98x0.95mm_HandSolder, symbol Device:R
- removed R1: 180k ohm, Resistor_SMD:R_0603_1608Metric_Pad0.98x0.95mm_HandSolder, symbol Device:R
- removed R12, R20 (x2), R21 (x2): 100k, Resistor_SMD:R_0603_1608Metric_Pad0.98x0.95mm_HandSolder, symbol Device:R
- removed R13, R25: 120R, Resistor_SMD:R_0603_1608Metric_Pad0.98x0.95mm_HandSolder, symbol Device:R
- removed R18 (x2), R19 (x2), R?: 100E, Resistor_SMD:R_0603_1608Metric_Pad0.98x0.95mm_HandSolder, symbol Device:R
- removed R2: 20k ohm, Resistor_SMD:R_0603_1608Metric_Pad0.98x0.95mm_HandSolder, symbol Device:R
- removed R2: 56k, Resistor_SMD:R_0603_1608Metric_Pad0.98x0.95mm_HandSolder, symbol Device:R
- removed R3: 698k ohm, Resistor_SMD:R_0603_1608Metric_Pad0.98x0.95mm_HandSolder, symbol Device:R
- removed R5: 100R, Resistor_SMD:R_0603_1608Metric_Pad0.98x0.95mm_HandSolder, symbol Device:R
- removed R?: 3M, Resistor_SMD:R_0603_1608Metric_Pad0.98x0.95mm_HandSolder, symbol Device:R
- removed R? (x7): 0R, Resistor_SMD:R_0603_1608Metric_Pad0.98x0.95mm_HandSolder, symbol Device:R
- removed R?: 1k, Resistor_SMD:R_0603_1608Metric_Pad0.98x0.95mm_HandSolder, symbol Device:R
- removed U2: LP2985-3.3, Package_TO_SOT_SMD:SOT-23-5, symbol Regulator_Linear:LP2985-3.3
- removed U3: TPS563200, Package_TO_SOT_SMD:SOT-23-6, symbol Regulator_Switching:TPS563200
- removed U4: STM32G0B1CBTx, Package_QFP:LQFP-48_7x7mm_P0.5mm, symbol MCU_ST_STM32G0:STM32G0B1CBTx
- removed U7: TJA1051T-3, Package_SO:SOIC-8_3.9x4.9mm_P1.27mm, symbol Interface_CAN_LIN:TJA1051T-3
- removed U?: MAX485E, MAX485ESA_T.kicad_mod files:SOIC127P600X175-8N, symbol Interface_UART:MAX485E
Connections:
- no-connect marks 51 -> 0
Other:
- added sheet Ble Unit (Ble.kicad_sch)
- added sheet Buzzer Unit  (Buzzer Unit.kicad_sch)
- added sheet Ina_228 (Ina_228.kicad_sch)
- added sheet POWER_UNIT (POWER.kicad_sch)
- added sheet STM32MCU (untitled.kicad_sch)
- added sheet Tranceiver (Tranceiver.kicad_sch)
- note removed: "BLE Unit"
- note removed: "Buzzer Unit"
- note removed: "LDO3.3V"
- note removed: "POWER SUPPLY UNIT"
- note removed: "STM32MCU"
- note removed: "TPS563203"
- note removed: "Transceiver"
- moved on the sheet: H1, H2, H3, H4, H5, H6
