File: SOC DISPLAY.kicad_sch (KiCad schematic)
At the start: 6 parts

Commit message: Ve
Other:
- removed sheet Ina_228
Changed lines of the file:
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@@
-    )
-  )
-  (sheet (at 124.46 110.49) (size 26.67 15.24) (fields_autoplaced)
-    (stroke (width 0.1524) (type solid))
-    (fill (color 0 0 0 0.0000))
-    (property "Sheetname" "Ina_228" (at 124.46 109.7784 0)
-      (effects (font (size 1.27 1.27)) (justify left bottom))
-    )
-    (property "Sheetfile" "Ina_228.kicad_sch" (at 124.46 126.3146 0)
-      (effects (font (size 1.27 1.27)) (justify left top))
-    )
-    (instances
-      (project "SOC DISPLAY"
-        (path "/9f7696f8-e9fa-4362-b2ca-5dde3355ad01" (page "7"))
-      )
     )
   )

Commit message: add text
Other:
- note added: "SECOND_PROJECT(SOC_DISPLAY+BLE_MODULE)"
Changed lines of the file:
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@@
     (fill (type none))
+  )
+  (text "SECOND_PROJECT(SOC_DISPLAY+BLE_MODULE)" (at 74.93 22.86 0)
+    (effects (font (size 5 5) (thickness 0.6) bold) (justify left bottom))
   )
   (symbol (lib_id "Mechanical:MountingHole") (at 256.54 124.46 0) (unit 1)

Commit message: Sch
Other:
- added sheet Ina_228 (Ina.kicad_sch)
Changed lines of the file:
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@@
+    )
+  )
+  (sheet (at 109.22 111.76) (size 48.26 17.78) (fields_autoplaced)
+    (stroke (width 0.1524) (type solid))
+    (fill (color 0 0 0 0.0000))
+    (property "Sheetname" "Ina_228" (at 109.22 111.0484 0)
+      (effects (font (size 1.27 1.27)) (justify left bottom))
+    )
+    (property "Sheetfile" "Ina.kicad_sch" (at 109.22 130.1246 0)
+      (effects (font (size 1.27 1.27)) (justify left top))
+    )
+    (instances
+      (project "SOC DISPLAY"
+        (path "/9f7696f8-e9fa-4362-b2ca-5dde3355ad01" (page "7"))
+      )
     )
   )
