File: POWER.kicad_sch (KiCad schematic)
At the start: 23 parts, among them IC2 LM5164QDDATQ1, U2 LP2985-3.3, U3 TPS563200

Commit message: Designator
Parts:
- 100k1: value R24 -> 100K
- 1M1: value R22 -> 1M
- 332k1: value R23 -> 332K
Changed lines of the file:
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@@
         )
         (path "/9f7696f8-e9fa-4362-b2ca-5dde3355ad01/f6af75e3-ef65-47cd-959b-72e6fa5f8f61"
-          (reference "C?") (unit 1)
+          (reference "C109") (unit 1)
         )
       )
@@
       (effects (font (size 1.27 1.27)) (justify left))
     )
-    (property "Value" "R22" (at 95.25 96.52 0)
+    (property "Value" "1M" (at 95.25 96.52 0)
       (effects (font (size 1.27 1.27)) (justify left))
     )
@@
         )
         (path "/9f7696f8-e9fa-4362-b2ca-5dde3355ad01/f6af75e3-ef65-47cd-959b-72e6fa5f8f61"
-          (reference "1M?") (unit 1)
+          (reference "R102") (unit 1)
         )
       )
@@
         )
         (path "/9f7696f8-e9fa-4362-b2ca-5dde3355ad01/f6af75e3-ef65-47cd-959b-72e6fa5f8f61"
-          (reference "#PWR027") (unit 1)
+          (reference "#PWR0102") (unit 1)
         )
       )
@@
         )
         (path "/9f7696f8-e9fa-4362-b2ca-5dde3355ad01/f6af75e3-ef65-47cd-959b-72e6fa5f8f61"
-          (reference "R?") (unit 1)
+          (reference "R104") (unit 1)
         )
       )
@@
         )
         (path "/9f7696f8-e9fa-4362-b2ca-5dde3355ad01/f6af75e3-ef65-47cd-959b-72e6fa5f8f61"
-          (reference "R?") (unit 1)
+          (reference "R108") (unit 1)
         )
       )
@@
         )
         (path "/9f7696f8-e9fa-4362-b2ca-5dde3355ad01/f6af75e3-ef65-47cd-959b-72e6fa5f8f61"
-          (reference "C?") (unit 1)
+          (reference "C102") (unit 1)
         )
       )
@@
         )
         (path "/9f7696f8-e9fa-4362-b2ca-5dde3355ad01/f6af75e3-ef65-47cd-959b-72e6fa5f8f61"
-          (reference "#PWR029") (unit 1)
+          (reference "#PWR0104") (unit 1)
         )
       )
@@
       (effects (font (size 1.27 1.27)) (justify left))
     )
-    (property "Value" "R23" (at 95.25 104.14 0)
+    (property "Value" "332K" (at 95.25 104.14 0)
       (effects (font (size 1.27 1.27)) (justify left))
     )
@@
         )
         (path "/9f7696f8-e9fa-4362-b2ca-5dde3355ad01/f6af75e3-ef65-47cd-959b-72e6fa5f8f61"
-          (reference "332k?") (unit 1)
+          (reference "R103") (unit 1)
         )
       )
@@
   (symbol (lib_id "Device:C") (at 170.18 66.04 0) (unit 1)
     (in_bom yes) (on_board yes) (dnp no)
-    (property "Reference" "C1" (at 165.1 66.04 0)
+    (property "Reference" "C1" (at 163.83 66.04 0)
       (effects (font (size 1.27 1.27)) (justify left))
     )
@@
         )
         (path "/9f7696f8-e9fa-4362-b2ca-5dde3355ad01/f6af75e3-ef65-47cd-959b-72e6fa5f8f61"
-          (reference "C?") (unit 1)
+          (reference "C105") (unit 1)
         )
       )
@@
         )
         (path "/9f7696f8-e9fa-4362-b2ca-5dde3355ad01/f6af75e3-ef65-47cd-959b-72e6fa5f8f61"
-          (reference "C?") (unit 1)
+          (reference "C110") (unit 1)
         )
       )
@@
   (symbol (lib_id "Device:C") (at 107.95 69.85 90) (unit 1)
     (in_bom yes) (on_board yes) (dnp no)
-    (property "Reference" "C2" (at 107.95 67.31 90)
+    (property "Reference" "C2" (at 107.95 66.04 90)
       (effects (font (size 1.27 1.27)))
     )
@@
         )
         (path "/9f7696f8-e9fa-4362-b2ca-5dde3355ad01/f6af75e3-ef65-47cd-959b-72e6fa5f8f61"
-          (reference "C?") (unit 1)
+          (reference "C101") (unit 1)
         )
       )
@@
   (symbol (lib_id "Device:C") (at 171.45 95.25 90) (unit 1)
     (in_bom yes) (on_board yes) (dnp no)
-    (property "Reference" "C4" (at 168.91 95.25 0)
+    (property "Reference" "C4" (at 167.64 93.98 90)
       (effects (font (size 1.27 1.27)) (justify left))
     )
@@
         )
         (path "/9f7696f8-e9fa-4362-b2ca-5dde3355ad01/f6af75e3-ef65-47cd-959b-72e6fa5f8f61"
-          (reference "C?") (unit 1)
+          (reference "C106") (unit 1)
         )
       )
@@
         )
         (path "/9f7696f8-e9fa-4362-b2ca-5dde3355ad01/f6af75e3-ef65-47cd-959b-72e6fa5f8f61"
-          (reference "C?") (unit 1)
+          (reference "C104") (unit 1)
         )
       )
@@
         )
         (path "/9f7696f8-e9fa-4362-b2ca-5dde3355ad01/f6af75e3-ef65-47cd-959b-72e6fa5f8f61"
-          (reference "R?") (unit 1)
+          (reference "R106") (unit 1)
         )
       )
@@
         )
         (path "/9f7696f8-e9fa-4362-b2ca-5dde3355ad01/f6af75e3-ef65-47cd-959b-72e6fa5f8f61"
-          (reference "U?") (unit 1)
+          (reference "U101") (unit 1)
         )
       )
@@
         )
         (path "/9f7696f8-e9fa-4362-b2ca-5dde3355ad01/f6af75e3-ef65-47cd-959b-72e6fa5f8f61"
-          (reference "L?") (unit 1)
+          (reference "L102") (unit 1)
         )
       )
@@
         )
         (path "/9f7696f8-e9fa-4362-b2ca-5dde3355ad01/f6af75e3-ef65-47cd-959b-72e6fa5f8f61"
-          (reference "IC?") (unit 1)
+          (reference "IC101") (unit 1)
         )
       )
@@
   (symbol (lib_id "Device:L") (at 96.52 66.04 90) (unit 1)
     (in_bom yes) (on_board yes) (dnp no)
-    (property "Reference" "L1" (at 93.98 64.77 90)
+    (property "Reference" "L1" (at 95.25 63.5 90)
       (effects (font (size 1.27 1.27)))
     )
@@
         )
         (path "/9f7696f8-e9fa-4362-b2ca-5dde3355ad01/f6af75e3-ef65-47cd-959b-72e6fa5f8f61"
-          (reference "L?") (unit 1)
+          (reference "L101") (unit 1)
         )
       )
@@
         )
         (path "/9f7696f8-e9fa-4362-b2ca-5dde3355ad01/f6af75e3-ef65-47cd-959b-72e6fa5f8f61"
-          (reference "#PWR030") (unit 1)
+          (reference "#PWR0105") (unit 1)
         )
       )
@@
         )
         (path "/9f7696f8-e9fa-4362-b2ca-5dde3355ad01/f6af75e3-ef65-47cd-959b-72e6fa5f8f61"
-          (reference "R?") (unit 1)
+          (reference "R107") (unit 1)
         )
       )
@@
         )
         (path "/9f7696f8-e9fa-4362-b2ca-5dde3355ad01/f6af75e3-ef65-47cd-959b-72e6fa5f8f61"
-          (reference "C?") (unit 1)
+          (reference "C103") (unit 1)
         )
       )
@@
         )
         (path "/9f7696f8-e9fa-4362-b2ca-5dde3355ad01/f6af75e3-ef65-47cd-959b-72e6fa5f8f61"
-          (reference "C?") (unit 1)
+          (reference "C108") (unit 1)
         )
       )
@@
         )
         (path "/9f7696f8-e9fa-4362-b2ca-5dde3355ad01/f6af75e3-ef65-47cd-959b-72e6fa5f8f61"
-          (reference "#PWR032") (unit 1)
+          (reference "#PWR0107") (unit 1)
         )
       )
@@
       (effects (font (size 1.27 1.27)) (justify left))
     )
-    (property "Value" "R24" (at 113.03 105.41 0)
+    (property "Value" "100K" (at 113.03 105.41 0)
       (effects (font (size 1.27 1.27)) (justify left))
     )
@@
         )
         (path "/9f7696f8-e9fa-4362-b2ca-5dde3355ad01/f6af75e3-ef65-47cd-959b-72e6fa5f8f61"
-          (reference "100k?") (unit 1)
+          (reference "R105") (unit 1)
         )
       )
@@
         )
         (path "/9f7696f8-e9fa-4362-b2ca-5dde3355ad01/f6af75e3-ef65-47cd-959b-72e6fa5f8f61"
-          (reference "#PWR031") (unit 1)
+          (reference "#PWR0106") (unit 1)
         )
       )
@@
         )
         (path "/9f7696f8-e9fa-4362-b2ca-5dde3355ad01/f6af75e3-ef65-47cd-959b-72e6fa5f8f61"
-          (reference "C?") (unit 1)
+          (reference "C107") (unit 1)
         )
       )
@@
         )
         (path "/9f7696f8-e9fa-4362-b2ca-5dde3355ad01/f6af75e3-ef65-47cd-959b-72e6fa5f8f61"
-          (reference "U?") (unit 1)
+          (reference "U102") (unit 1)
         )
       )
@@
         )
         (path "/9f7696f8-e9fa-4362-b2ca-5dde3355ad01/f6af75e3-ef65-47cd-959b-72e6fa5f8f61"
-          (reference "#PWR028") (unit 1)
+          (reference "#PWR0103") (unit 1)
         )
       )
@@
         )
         (path "/9f7696f8-e9fa-4362-b2ca-5dde3355ad01/f6af75e3-ef65-47cd-959b-72e6fa5f8f61"
-          (reference "#PWR034") (unit 1)
+          (reference "#PWR0109") (unit 1)
         )
       )
@@
         )
         (path "/9f7696f8-e9fa-4362-b2ca-5dde3355ad01/f6af75e3-ef65-47cd-959b-72e6fa5f8f61"
-          (reference "#PWR026") (unit 1)
+          (reference "#PWR0101") (unit 1)
         )
       )
@@
         )
         (path "/9f7696f8-e9fa-4362-b2ca-5dde3355ad01/f6af75e3-ef65-47cd-959b-72e6fa5f8f61"
-          (reference "R?") (unit 1)
+          (reference "R101") (unit 1)
         )
       )
@@
         )
         (path "/9f7696f8-e9fa-4362-b2ca-5dde3355ad01/f6af75e3-ef65-47cd-959b-72e6fa5f8f61"
-          (reference "#PWR033") (unit 1)
-        )
-      )
+          (reference "#PWR0108") (unit 1)
+        )
+      )
