File: POWER.kicad_sch (KiCad schematic)
At the start: 23 parts, among them IC2 LM5164QDDATQ1, U2 LP2985-3.3, U3 TPS563200

Commit message: giga
Parts:
- added R5, R7, R8: 0R, Resistor_SMD:R_0603_1608Metric_Pad0.98x0.95mm_HandSolder, symbol Device:R
- 332k1: value 332K -> 300K
- C1, C2, C4: footprint Capacitor_SMD:C_0805_2012Metric_Pad1.18x1.45mm_HandSolder -> Capacitor_SMD:C_0603_1608Metric_Pad1.08x0.95mm_HandSolder
- C5: footprint Capacitor_SMD:C_0402_1005Metric_Pad0.74x0.62mm_HandSolder -> Capacitor_SMD:C_0603_1608Metric_Pad1.08x0.95mm_HandSolder
- L1: footprint Inductor_SMD:L_0805_2012Metric_Pad1.15x1.40mm_HandSolder -> LIB_1267AY-101M=P3.kicad_mod files:1267AY6R8NP3
- L1: footprint Inductor_SMD:L_0402_1005Metric_Pad0.77x0.64mm_HandSolder -> Library:INR33
- R3: value 698k ohm -> 700k ohm
Connections:
- net 12V: now also R5.2, R7.2; no longer C3.1, C3.1, C4.2, L1.2, R1.1
- net 5V: now also R8.2; no longer L1.2, R2.2
- net GND: now also IC2.9 (EP)
- new net 12Vcc: C3.1, C3.1, C4.2, L1.2, R1.1, R5.1, R7.1
- new net 5Vcc: L1.2, R2.2, R8.1
- no-connect marks 2 -> 1
