File: POWER.kicad_sch (KiCad schematic)
At the start: 26 parts, among them IC2 LM5164QDDATQ1, U2 LP2985-3.3, U3 TPS563200

Commit message: new
Changed lines of the file:
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@@
   (junction (at 120.65 58.42) (diameter 0) (color 0 0 0 0)
   )
+  (junction (at 140.97 64.77) (diameter 0) (color 0 0 0 0)
+  )
   (no_connect (at 156.21 96.52))
+  (wire (pts (xy 140.97 64.77) (xy 142.24 64.77))
+    (stroke (width 0) (type default))
+  )
   (wire (pts (xy 195.58 60.96) (xy 190.5 60.96))
     (stroke (width 0) (type default))
@@
     (stroke (width 0) (type default))
   )
-  (wire (pts (xy 139.7 64.77) (xy 142.24 64.77))
+  (wire (pts (xy 139.7 64.77) (xy 140.97 64.77))
     (stroke (width 0) (type default))
   )
@@
   )
   (wire (pts (xy 167.64 60.96) (xy 167.64 62.23))
+    (stroke (width 0) (type default))
+  )
+  (wire (pts (xy 140.97 67.31) (xy 140.97 64.77))
     (stroke (width 0) (type default))
   )
@@
     (fill (type none))
   )
-  (rectangle (start 83.82 52.07) (end 151.13 74.93)
+  (rectangle (start 83.82 50.8) (end 151.13 74.93)
     (stroke (width 0.2) (type dot) (color 56 179 255 1))
     (fill (type none))
   )
-  (rectangle (start 152.4 52.07) (end 217.17 74.93)
+  (rectangle (start 152.4 50.8) (end 217.17 74.93)
     (stroke (width 0.2) (type dot) (color 56 179 255 1))
     (fill (type none))
@@
     (effects (font (size 1.27 1.27) (thickness 0.254) bold) (justify right bottom))
   )
-  (text "POWER SUPPLY UNIT \n\n\n" (at 80.01 50.8 0)
+  (text "POWER SUPPLY UNIT \n\n\n" (at 113.03 48.26 0)
     (effects (font (size 2.5 2.5) (thickness 0.65) bold) (justify left bottom))
   )
@@
   (label "GND" (at 180.34 72.39 0) (fields_autoplaced)
     (effects (font (size 1.27 1.27)) (justify left bottom))
-  )
-  (label "12V" (at 140.97 64.77 0) (fields_autoplaced)
-    (effects (font (size 1.27 1.27)) (justify left bottom))
-  )
-  (label "12V" (at 120.65 57.15 180) (fields_autoplaced)
-    (effects (font (size 1.27 1.27)) (justify right bottom))
   )
   (global_label "VBST" (shape input) (at 101.6 69.85 180) (fields_autoplaced)
@@
       (effects (font (size 1.27 1.27)) (justify left) hide)
     )
+  )
+  (global_label "12V" (shape input) (at 140.97 67.31 0) (fields_autoplaced)
+    (effects (font (size 1.27 1.27)) (justify left))
+    (property "Intersheetrefs" "${INTERSHEET_REFS}" (at 147.3834 67.31 0)
+      (effects (font (size 1.27 1.27)) (justify left) hide)
+    )
+  )
+  (global_label "12V" (shape input) (at 120.65 57.15 90) (fields_autoplaced)
+    (effects (font (size 1.27 1.27)) (justify left))
+    (property "Intersheetrefs" "${INTERSHEET_REFS}" (at 120.65 50.7366 90)
+      (effects (font (size 1.27 1.27)) (justify left) hide)
+    )

Commit message: giga
Parts:
- renumbered R5 to R105, R7 to R107, R8 to R108
