File: Ble.kicad_sch (KiCad schematic)
At the start: 2 parts, among them IC1 CM BLE

Commit message: some
Parts:
- removed R?: 1k, Resistor_SMD:R_0603_1608Metric_Pad0.98x0.95mm_HandSolder, symbol Device:R
Connections:
- net RX: now also IC1.10 (P10)
- net TX: no longer IC1.10 (P10)
Changed lines of the file:
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@@
   (junction (at 168.91 86.36) (diameter 0) (color 0 0 0 0)
-  )
-  (junction (at 127 88.9) (diameter 0) (color 0 0 0 0)
   )
   (junction (at 168.91 106.68) (diameter 0) (color 0 0 0 0)
@@
   )
   (junction (at 168.91 96.52) (diameter 0) (color 0 0 0 0)
-  )
-  (junction (at 129.54 88.9) (diameter 0) (color 0 0 0 0)
   )
   (junction (at 168.91 113.03) (diameter 0) (color 0 0 0 0)
@@
     (stroke (width 0) (type default))
   )
-  (wire (pts (xy 119.38 88.9) (xy 127 88.9))
-    (stroke (width 0) (type default))
-  )
-  (wire (pts (xy 127 88.9) (xy 129.54 88.9))
+  (wire (pts (xy 124.46 88.9) (xy 129.54 88.9))
     (stroke (width 0) (type default))
   )
@@
   )
   (wire (pts (xy 168.91 73.66) (xy 168.91 76.2))
-    (stroke (width 0) (type default))
-  )
-  (wire (pts (xy 129.54 88.9) (xy 129.54 91.44))
     (stroke (width 0) (type default))
   )
@@
   )
   (wire (pts (xy 128.27 93.98) (xy 128.27 113.03))
+    (stroke (width 0) (type default))
+  )
+  (wire (pts (xy 129.54 91.44) (xy 124.46 91.44))
     (stroke (width 0) (type default))
   )
@@
     (stroke (width 0) (type default))
   )
-  (wire (pts (xy 127 88.9) (xy 127 91.44))
-    (stroke (width 0) (type default))
-  )
   (rectangle (start 111.76 55.88) (end 179.07 124.46)
     (stroke (width 0) (type dash_dot_dot))
@@
     (effects (font (size 1.27 1.27)) (justify left bottom))
   )
-  (label "RX" (at 119.38 91.44 180) (fields_autoplaced)
+  (label "RX" (at 124.46 91.44 180) (fields_autoplaced)
     (effects (font (size 1.27 1.27)) (justify right bottom))
   )
@@
     (effects (font (size 1.27 1.27)) (justify right bottom))
   )
-  (label "TX" (at 119.38 88.9 180) (fields_autoplaced)
+  (label "TX" (at 124.46 88.9 180) (fields_autoplaced)
     (effects (font (size 1.27 1.27)) (justify right bottom))
   )
@@
         )
       )
-    )
-  )
-  (symbol (lib_id "Device:R") (at 123.19 91.44 90) (unit 1)
-    (in_bom yes) (on_board yes) (dnp no)
-    (property "Reference" "R?" (at 123.19 93.98 90)
-      (effects (font (size 1.27 1.27)))
-    )
-    (property "Value" "1k" (at 123.19 91.44 90)
-      (effects (font (size 1.27 1.27)))
-    )
-    (property "Footprint" "Resistor_SMD:R_0603_1608Metric_Pad0.98x0.95mm_HandSolder" (at 123.19 93.218 90)
-      (effects (font (size 1.27 1.27)) hide)
-    )
-    (property "Datasheet" "~" (at 123.19 91.44 0)
-      (effects (font (size 1.27 1.27)) hide)
-    )
-    (pin "1")
-    (pin "2")
-    (instances
-      (project "SOC 2"
-        (path "/61c20a78-9f1a-4b1a-a5d9-ab1a8f753f68"
-          (reference "R?") (unit 1)
-        )
-      )
-      (project "SOC DISPLAY"
-        (path "/9f7696f8-e9fa-4362-b2ca-5dde3355ad01"
-          (reference "R2") (unit 1)
-        )
-        (path "/9f7696f8-e9fa-4362-b2ca-5dde3355ad01/3c4c5daf-1dcb-46b8-a7a7-925b6fcdbaca"
-          (reference "R501") (unit 1)
-        )
-      )
