File: untitled.kicad_sch (KiCad schematic)
At the start: 30 parts, among them J2 PRG, J3 OLED, U4 STM32G0B1CBTx

Commit message: giga
Parts:
- C1: footprint Capacitor_SMD:C_0805_2012Metric_Pad1.18x1.45mm_HandSolder -> Capacitor_SMD:C_0603_1608Metric_Pad1.08x0.95mm_HandSolder
Changed lines of the file:
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@@
         )
         (path "/9f7696f8-e9fa-4362-b2ca-5dde3355ad01/04eef66b-5e57-42e7-9448-b3758ef8edd2"
-          (reference "R205") (unit 1)
+          (reference "R16") (unit 1)
         )
       )
@@
         )
         (path "/9f7696f8-e9fa-4362-b2ca-5dde3355ad01/04eef66b-5e57-42e7-9448-b3758ef8edd2"
-          (reference "#PWR0210") (unit 1)
+          (reference "#PWR020") (unit 1)
         )
       )
@@
         )
         (path "/9f7696f8-e9fa-4362-b2ca-5dde3355ad01/04eef66b-5e57-42e7-9448-b3758ef8edd2"
-          (reference "J201") (unit 1)
+          (reference "J1") (unit 1)
         )
       )
@@
         )
         (path "/9f7696f8-e9fa-4362-b2ca-5dde3355ad01/04eef66b-5e57-42e7-9448-b3758ef8edd2"
-          (reference "#PWR0202") (unit 1)
+          (reference "#PWR012") (unit 1)
         )
       )
@@
         )
         (path "/9f7696f8-e9fa-4362-b2ca-5dde3355ad01/04eef66b-5e57-42e7-9448-b3758ef8edd2"
-          (reference "R202") (unit 1)
+          (reference "R13") (unit 1)
         )
       )
@@
         )
         (path "/9f7696f8-e9fa-4362-b2ca-5dde3355ad01/04eef66b-5e57-42e7-9448-b3758ef8edd2"
-          (reference "R216") (unit 1)
+          (reference "R27") (unit 1)
         )
       )
@@
         )
         (path "/9f7696f8-e9fa-4362-b2ca-5dde3355ad01/04eef66b-5e57-42e7-9448-b3758ef8edd2"
-          (reference "R218") (unit 1)
+          (reference "R29") (unit 1)
         )
       )
@@
         )
         (path "/9f7696f8-e9fa-4362-b2ca-5dde3355ad01/04eef66b-5e57-42e7-9448-b3758ef8edd2"
-          (reference "U202") (unit 1)
+          (reference "U4") (unit 1)
         )
       )
@@
         )
         (path "/9f7696f8-e9fa-4362-b2ca-5dde3355ad01/04eef66b-5e57-42e7-9448-b3758ef8edd2"
-          (reference "J203") (unit 1)
+          (reference "J3") (unit 1)
         )
       )
@@
         )
         (path "/9f7696f8-e9fa-4362-b2ca-5dde3355ad01/04eef66b-5e57-42e7-9448-b3758ef8edd2"
-          (reference "R217") (unit 1)
+          (reference "R28") (unit 1)
         )
       )
@@
         )
         (path "/9f7696f8-e9fa-4362-b2ca-5dde3355ad01/04eef66b-5e57-42e7-9448-b3758ef8edd2"
-          (reference "R207") (unit 1)
+          (reference "R18") (unit 1)
         )
       )
@@
         )
         (path "/9f7696f8-e9fa-4362-b2ca-5dde3355ad01/04eef66b-5e57-42e7-9448-b3758ef8edd2"
-          (reference "#PWR0204") (unit 1)
+          (reference "#PWR014") (unit 1)
         )
       )
@@
         )
         (path "/9f7696f8-e9fa-4362-b2ca-5dde3355ad01/04eef66b-5e57-42e7-9448-b3758ef8edd2"
-          (reference "#PWR0203") (unit 1)
+          (reference "#PWR013") (unit 1)
         )
       )
@@
         )
         (path "/9f7696f8-e9fa-4362-b2ca-5dde3355ad01/04eef66b-5e57-42e7-9448-b3758ef8edd2"
-          (reference "#PWR0206") (unit 1)
+          (reference "#PWR016") (unit 1)
         )
       )
@@
         )
         (path "/9f7696f8-e9fa-4362-b2ca-5dde3355ad01/04eef66b-5e57-42e7-9448-b3758ef8edd2"
-          (reference "R215") (unit 1)
+          (reference "R26") (unit 1)
         )
       )
@@
         )
         (path "/9f7696f8-e9fa-4362-b2ca-5dde3355ad01/04eef66b-5e57-42e7-9448-b3758ef8edd2"
-          (reference "#PWR0208") (unit 1)
+          (reference "#PWR018") (unit 1)
         )
       )
@@
         )
         (path "/9f7696f8-e9fa-4362-b2ca-5dde3355ad01/04eef66b-5e57-42e7-9448-b3758ef8edd2"
-          (reference "#PWR0201") (unit 1)
+          (reference "#PWR011") (unit 1)
         )
       )
@@
         )
         (path "/9f7696f8-e9fa-4362-b2ca-5dde3355ad01/04eef66b-5e57-42e7-9448-b3758ef8edd2"
-          (reference "#PWR0207") (unit 1)
+          (reference "#PWR017") (unit 1)
         )
       )
@@
         )
         (path "/9f7696f8-e9fa-4362-b2ca-5dde3355ad01/04eef66b-5e57-42e7-9448-b3758ef8edd2"
-          (reference "J204") (unit 1)
+          (reference "J4") (unit 1)
         )
       )
@@
         )
         (path "/9f7696f8-e9fa-4362-b2ca-5dde3355ad01/04eef66b-5e57-42e7-9448-b3758ef8edd2"
-          (reference "#PWR0209") (unit 1)
+          (reference "#PWR019") (unit 1)
         )
       )
@@
         )
         (path "/9f7696f8-e9fa-4362-b2ca-5dde3355ad01/04eef66b-5e57-42e7-9448-b3758ef8edd2"
-          (reference "R206") (unit 1)
+          (reference "R17") (unit 1)
         )
       )
@@
         )
         (path "/9f7696f8-e9fa-4362-b2ca-5dde3355ad01/04eef66b-5e57-42e7-9448-b3758ef8edd2"
-          (reference "R209") (unit 1)
+          (reference "R20") (unit 1)
         )
       )
@@
         )
         (path "/9f7696f8-e9fa-4362-b2ca-5dde3355ad01/04eef66b-5e57-42e7-9448-b3758ef8edd2"
-          (reference "R210") (unit 1)
+          (reference "R21") (unit 1)
         )
       )
@@
         )
         (path "/9f7696f8-e9fa-4362-b2ca-5dde3355ad01/04eef66b-5e57-42e7-9448-b3758ef8edd2"
-          (reference "J205") (unit 1)
+          (reference "J5") (unit 1)
         )
       )
@@
         )
         (path "/9f7696f8-e9fa-4362-b2ca-5dde3355ad01/04eef66b-5e57-42e7-9448-b3758ef8edd2"
-          (reference "R214") (unit 1)
+          (reference "R25") (unit 1)
         )
       )
@@
       (effects (font (size 1.27 1.27)) (justify left))
     )
-    (property "Footprint" "Capacitor_SMD:C_0805_2012Metric_Pad1.18x1.45mm_HandSolder" (at 145.7452 139.7 0)
+    (property "Footprint" "Capacitor_SMD:C_0603_1608Metric_Pad1.08x0.95mm_HandSolder" (at 145.7452 139.7 0)
       (effects (font (size 1.27 1.27)) hide)
     )
@@
         )
         (path "/9f7696f8-e9fa-4362-b2ca-5dde3355ad01/04eef66b-5e57-42e7-9448-b3758ef8edd2"
-          (reference "C202") (unit 1)
+          (reference "C12") (unit 1)
         )
       )
@@
       (effects (font (size 1.27 1.27)) (justify left))
     )
-    (property "Footprint" "Capacitor_SMD:C_0805_2012Metric_Pad1.18x1.45mm_HandSolder" (at 97.4852 134.62 0)
+    (property "Footprint" "Capacitor_SMD:C_0603_1608Metric_Pad1.08x0.95mm_HandSolder" (at 97.4852 134.62 0)
       (effects (font (size 1.27 1.27)) hide)
     )
@@
         )
         (path "/9f7696f8-e9fa-4362-b2ca-5dde3355ad01/04eef66b-5e57-42e7-9448-b3758ef8edd2"
-          (reference "C201") (unit 1)
+          (reference "C11") (unit 1)
         )
       )
@@
         )
         (path "/9f7696f8-e9fa-4362-b2ca-5dde3355ad01/04eef66b-5e57-42e7-9448-b3758ef8edd2"
-          (reference "R203") (unit 1)
+          (reference "R14") (unit 1)
         )
       )
@@
         )
         (path "/9f7696f8-e9fa-4362-b2ca-5dde3355ad01/04eef66b-5e57-42e7-9448-b3758ef8edd2"
-          (reference "J202") (unit 1)
+          (reference "J2") (unit 1)
         )
       )
@@
         )
         (path "/9f7696f8-e9fa-4362-b2ca-5dde3355ad01/04eef66b-5e57-42e7-9448-b3758ef8edd2"
-          (reference "#PWR0205") (unit 1)
+          (reference "#PWR015") (unit 1)
         )
       )
@@
         )
         (path "/9f7696f8-e9fa-4362-b2ca-5dde3355ad01/04eef66b-5e57-42e7-9448-b3758ef8edd2"
-          (reference "R213") (unit 1)
+          (reference "R24") (unit 1)
         )
       )
@@
         )
         (path "/9f7696f8-e9fa-4362-b2ca-5dde3355ad01/04eef66b-5e57-42e7-9448-b3758ef8edd2"
-          (reference "R208") (unit 1)
+          (reference "R19") (unit 1)
         )
       )
@@
         )
         (path "/9f7696f8-e9fa-4362-b2ca-5dde3355ad01/04eef66b-5e57-42e7-9448-b3758ef8edd2"
-          (reference "R212") (unit 1)
+          (reference "R23") (unit 1)
         )
       )
@@
         )
         (path "/9f7696f8-e9fa-4362-b2ca-5dde3355ad01/04eef66b-5e57-42e7-9448-b3758ef8edd2"
-          (reference "E201") (unit 1)
+          (reference "E1") (unit 1)
         )
       )
@@
         )
         (path "/9f7696f8-e9fa-4362-b2ca-5dde3355ad01/04eef66b-5e57-42e7-9448-b3758ef8edd2"
-          (reference "R204") (unit 1)
+          (reference "R15") (unit 1)
         )
       )
@@
         )
         (path "/9f7696f8-e9fa-4362-b2ca-5dde3355ad01/04eef66b-5e57-42e7-9448-b3758ef8edd2"
-          (reference "U201") (unit 1)
+          (reference "U3") (unit 1)
         )
       )
@@
         )
         (path "/9f7696f8-e9fa-4362-b2ca-5dde3355ad01/04eef66b-5e57-42e7-9448-b3758ef8edd2"
-          (reference "R211") (unit 1)
+          (reference "R22") (unit 1)
         )
       )
@@
         )
         (path "/9f7696f8-e9fa-4362-b2ca-5dde3355ad01/04eef66b-5e57-42e7-9448-b3758ef8edd2"
-          (reference "F201") (unit 1)
+          (reference "F1") (unit 1)
         )
       )
@@
       (effects (font (size 1.27 1.27)) (justify left))
     )
-    (property "Footprint" "Capacitor_SMD:C_0805_2012Metric_Pad1.18x1.45mm_HandSolder" (at 150.8252 139.7 0)
+    (property "Footprint" "Capacitor_SMD:C_0603_1608Metric_Pad1.08x0.95mm_HandSolder" (at 150.8252 139.7 0)
       (effects (font (size 1.27 1.27)) hide)
     )
@@
         )
         (path "/9f7696f8-e9fa-4362-b2ca-5dde3355ad01/04eef66b-5e57-42e7-9448-b3758ef8edd2"
-          (reference "C203") (unit 1)
+          (reference "C13") (unit 1)
         )
       )
@@
         )
         (path "/9f7696f8-e9fa-4362-b2ca-5dde3355ad01/04eef66b-5e57-42e7-9448-b3758ef8edd2"
-          (reference "R201") (unit 1)
-        )
-      )
+          (reference "R12") (unit 1)
+        )
+      )
