File: untitled.kicad_sch (KiCad schematic)
At the start: 30 parts, among them J2 PRG, J3 OLED, U4 STM32G0B1CBTx

Commit message: new
Changed lines of the file:
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@@
     (effects (font (size 1.27 1.27)) (justify right bottom))
-  )
-  (label "12V" (at 173.99 92.71 90) (fields_autoplaced)
-    (effects (font (size 1.27 1.27)) (justify left bottom))
   )
   (label "RX" (at 137.16 81.28 0) (fields_autoplaced)
@@
       (effects (font (size 1.27 1.27)) (justify left) hide)
     )
+  )
+  (global_label "12V" (shape input) (at 173.99 92.71 90) (fields_autoplaced)
+    (effects (font (size 1.27 1.27)) (justify left))
+    (property "Intersheetrefs" "${INTERSHEET_REFS}" (at 173.99 86.2966 90)
+      (effects (font (size 1.27 1.27)) (justify left) hide)
+    )
