File: Buzzer Unit.kicad_sch (KiCad schematic)
At the start: 6 parts

Commit message: Hat
Changed lines of the file:
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@@
   (symbol (lib_id "Device:R") (at 119.38 100.33 0) (unit 1)
     (in_bom yes) (on_board yes) (dnp no)
-    (property "Reference" "R?" (at 121.92 99.06 0)
+    (property "Reference" "R?" (at 114.3 99.06 0)
       (effects (font (size 1.27 1.27)) (justify left))
     )
