File: SOC DISPLAY(1).kicad_pcb (KiCad board)
At the start: 2 copper layers, 47.2 x 46.7 mm, 70 parts, among them IC1 CM BLE, IC2 LM5164QDDATQ1, J1 PRG, J2 Conn_01x05_Socket, J3 OLED, J4 OLED, J5 Conn_01x02_Socket, Q1 NDT3055L, U1 STM32G0B1CBTx, U2 MAX485E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

Commit message: Hat
Parts:
- moved J4 41.0 mm to (114.6, 39.4), turned to 180 degrees
- moved J3 40.2 mm to (92.5, 58.7), turned to -90 degrees
- moved H5 32.7 mm to (135.6, 37.6)
- moved H6 31.7 mm to (135.6, 50.8)
- moved J2 23.4 mm to (130.6, 41.9)
- moved R7 0.21 mm to (98.3, 58.3)
Other:
- board size 47.2 x 46.7 mm -> 49.8 x 46.7 mm
Changed lines of the file:
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@@
   )
   (footprint "MountingHole:MountingHole_2.7mm_M2.5_ISO7380_Pad_TopBottom" (layer "F.Cu")
-    (at 166.37 58.42)
+    (at 135.636 50.8)
     (descr "Mounting Hole 2.7mm, M2.5, ISO7380")
     (tags "mounting hole 2.7mm m2.5 iso7380")
@@
     (property "ki_keywords" "R res resistor")
     (attr smd)
-    (fp_text reference "R13" (at -1.9285 0) (layer "F.SilkS")
+    (fp_text reference "R13" (at -1.8815 0) (layer "F.SilkS")
         (effects (font (size 0.3 0.3) (thickness 0.075) bold))
     )
@@
     (property "ki_keywords" "R res resistor")
     (attr smd)
-    (fp_text reference "R14" (at -1.949 0 180) (layer "F.SilkS")
+    (fp_text reference "R14" (at -1.8815 0 180) (layer "F.SilkS")
         (effects (font (size 0.3 0.3) (thickness 0.075) bold))
     )
@@
   )
   (footprint "TerminalBlock:TerminalBlock_bornier-4_P5.08mm" (layer "F.Cu")
-    (at 127.762 39.37 180)
+    (at 92.456 58.674 -90)
     (descr "simple 4-pin terminal block, pitch 5.08mm, revamped version of bornier4")
     (tags "terminal block bornier4")
@@
     (property "ki_keywords" "connector")
     (attr through_hole)
-    (fp_text reference "J3" (at 14.478 -4.318) (layer "F.SilkS")
+    (fp_text reference "J3" (at 14.478 -4.318 -270) (layer "F.SilkS")
         (effects (font (size 0.3 0.3) (thickness 0.075) bold))
     )
-    (fp_text value "OLED" (at 7.6 4.75) (layer "F.Fab")
+    (fp_text value "OLED" (at 7.6 4.75 -270) (layer "F.Fab")
         (effects (font (size 1 1) (thickness 0.15)))
     )
-    (fp_text user "${REFERENCE}" (at 7.62 0) (layer "F.Fab")
+    (fp_text user "${REFERENCE}" (at 7.62 0 -270) (layer "F.Fab")
         (effects (font (size 1 1) (thickness 0.15)))
     )
@@
     (fp_line (start 17.72 3.75) (end -2.43 3.75)
       (stroke (width 0.1) (type solid)) (layer "F.Fab"))
-    (pad "1" thru_hole rect (at 0 0 180) (size 3 3) (drill 1.52) (layers "*.Cu" "*.Mask")
+    (pad "1" thru_hole rect (at 0 0 270) (size 3 3) (drill 1.52) (layers "*.Cu" "*.Mask")
       (net 34 "5V") (pinfunction "Pin_1") (pintype "passive"))
-    (pad "2" thru_hole circle (at 5.08 0 180) (size 3 3) (drill 1.52) (layers "*.Cu" "*.Mask")
+    (pad "2" thru_hole circle (at 5.08 0 270) (size 3 3) (drill 1.52) (layers "*.Cu" "*.Mask")
       (net 78 "SDA_2") (pinfunction "Pin_2") (pintype "passive"))
-    (pad "3" thru_hole circle (at 10.16 0 180) (size 3 3) (drill 1.52) (layers "*.Cu" "*.Mask")
+    (pad "3" thru_hole circle (at 10.16 0 270) (size 3 3) (drill 1.52) (layers "*.Cu" "*.Mask")
       (net 88 "SCK_2") (pinfunction "Pin_3") (pintype "passive"))
-    (pad "4" thru_hole circle (at 15.24 0 180) (size 3 3) (drill 1.52) (layers "*.Cu" "*.Mask")
+    (pad "4" thru_hole circle (at 15.24 0 270) (size 3 3) (drill 1.52) (layers "*.Cu" "*.Mask")
       (net 4 "GND") (pinfunction "Pin_4") (pintype "passive"))
     (model "${KICAD6_3DMODEL_DIR}/TerminalBlock.3dshapes/TerminalBlock_bornier-4_P5.08mm.wrl"
@@
   )
   (footprint "TerminalBlock:TerminalBlock_bornier-4_P5.08mm" (layer "F.Cu")
-    (at 92.456 73.914 90)
+    (at 114.554 39.37 180)
     (descr "simple 4-pin terminal block, pitch 5.08mm, revamped version of bornier4")
     (tags "terminal block bornier4")
@@
     (property "ki_keywords" "connector")
     (attr through_hole)
-    (fp_text reference "J4" (at 11.938 4.318 180) (layer "F.SilkS")
+    (fp_text reference "J4" (at 8.382 -4.572 180) (layer "F.SilkS")
         (effects (font (size 0.3 0.3) (thickness 0.075) bold))
     )
-    (fp_text value "OLED" (at 7.6 4.75 90) (layer "F.Fab")
+    (fp_text value "OLED" (at 7.6 4.75) (layer "F.Fab")
         (effects (font (size 1 1) (thickness 0.15)))
     )
-    (fp_text user "${REFERENCE}" (at 7.62 0 90) (layer "F.Fab")
+    (fp_text user "${REFERENCE}" (at 7.62 0) (layer "F.Fab")
         (effects (font (size 1 1) (thickness 0.15)))
     )
@@
     (fp_line (start 17.72 3.75) (end -2.43 3.75)
       (stroke (width 0.1) (type solid)) (layer "F.Fab"))
-    (pad "1" thru_hole rect (at 0 0 90) (size 3 3) (drill 1.52) (layers "*.Cu" "*.Mask")
+    (pad "1" thru_hole rect (at 0 0 180) (size 3 3) (drill 1.52) (layers "*.Cu" "*.Mask")
       (net 34 "5V") (pinfunction "Pin_1") (pintype "passive"))
-    (pad "2" thru_hole circle (at 5.08 0 90) (size 3 3) (drill 1.52) (layers "*.Cu" "*.Mask")
+    (pad "2" thru_hole circle (at 5.08 0 180) (size 3 3) (drill 1.52) (layers "*.Cu" "*.Mask")
       (net 35 "SDA1") (pinfunction "Pin_2") (pintype "passive"))
-    (pad "3" thru_hole circle (at 10.16 0 90) (size 3 3) (drill 1.52) (layers "*.Cu" "*.Mask")
+    (pad "3" thru_hole circle (at 10.16 0 180) (size 3 3) (drill 1.52) (layers "*.Cu" "*.Mask")
       (net 36 "SCK") (pinfunction "Pin_3") (pintype "passive"))
-    (pad "4" thru_hole circle (at 15.24 0 90) (size 3 3) (drill 1.52) (layers "*.Cu" "*.Mask")
+    (pad "4" thru_hole circle (at 15.24 0 180) (size 3 3) (drill 1.52) (layers "*.Cu" "*.Mask")
       (net 4 "GND") (pinfunction "Pin_4") (pintype "passive"))
     (model "${KICAD6_3DMODEL_DIR}/TerminalBlock.3dshapes/TerminalBlock_bornier-4_P5.08mm.wrl"
@@
     (property "ki_keywords" "R res resistor")
     (attr smd)
-    (fp_text reference "R4" (at -0.1555 -1.016 180) (layer "F.SilkS")
+    (fp_text reference "R4" (at -1.9285 0 180) (layer "F.SilkS")
         (effects (font (size 0.3 0.3) (thickness 0.075) bold))
     )
@@
   )
   (footprint "Connector_JST:JST_PH_S5B-PH-K_1x05_P2.00mm_Horizontal" (layer "F.Cu")
-    (at 107.188 42.164 180)
+    (at 130.556 41.91 180)
     (descr "JST PH series connector, S5B-PH-K (http://www.jst-mfg.com/product/pdf/eng/ePH.pdf), generated with kicad-footprint-generator")
     (tags "connector JST PH top entry")
@@
     (property "ki_keywords" "R res resistor")
     (attr smd)
-    (fp_text reference "R17" (at 1.9285 0 -180) (layer "F.SilkS")
+    (fp_text reference "R17" (at 1.8815 0 -180) (layer "F.SilkS")
         (effects (font (size 0.3 0.3) (thickness 0.075) bold))
     )
@@
     (property "ki_keywords" "R res resistor")
     (attr smd)
-    (fp_text reference "R16" (at -1.9285 0 180) (layer "F.SilkS")
+    (fp_text reference "R16" (at -1.8815 0 180) (layer "F.SilkS")
         (effects (font (size 0.3 0.3) (thickness 0.075) bold))
     )
@@
   )
   (footprint "MountingHole:MountingHole_2.7mm_M2.5_ISO7380_Pad_TopBottom" (layer "F.Cu")
-    (at 166.37 48.768)
+    (at 135.636 37.592)
     (descr "Mounting Hole 2.7mm, M2.5, ISO7380")
     (tags "mounting hole 2.7mm m2.5 iso7380")
@@
   )
   (footprint "Resistor_SMD:R_0603_1608Metric_Pad0.98x0.95mm_HandSolder" (layer "F.Cu")
-    (at 98.298 58.5235 90)
+    (at 98.298 58.3165 90)
     (descr "Resistor SMD 0603 (1608 Metric), square (rectangular) end terminal, IPC_7351 nominal with elongated pad for handsoldering. (Body size source: IPC-SM-782 page 72, https://www.pcb-3d.com/wordpress/wp-content/uploads/ipc-sm-782a_amendment_1_and_2.pdf), generated with kicad-footprint-generator")
     (tags "resistor handsolder")
@@
     (property "ki_keywords" "R res resistor")
     (attr smd)
-    (fp_text reference "R7" (at -0.566752 -1.0095 90) (layer "F.SilkS")
+    (fp_text reference "R7" (at -1.8815 0 180) (layer "F.SilkS")
         (effects (font (size 0.3 0.3) (thickness 0.075) bold))
     )
@@
     (pad "1" connect circle (at 0 0) (size 4.5 4.5) (layers "B.Cu" "B.Mask"))
   )
-  (gr_rect (start 88.392 35.052) (end 135.636 81.788)
+  (gr_rect (start 88.392 35.052) (end 138.176 81.788)
     (stroke (width 0.05) (type default)) (fill none) (layer "Edge.Cuts"))
   (segment (start 105.3335 55.118) (end 105.3335 55.4485) (width 0.2) (layer "F.Cu") (net 92))
