File: Ina.kicad_sch (KiCad schematic)
At the start: 15 parts, among them J6 Conn_01x02_Pin, J7 Conn_01x02_Pin, U6 INA228AQDGSRQ1

Commit message: giga
Parts:
- renumbered C14 to C601, C15 to C602, C16 to C603, C17 to C604, J6 to J601, J7 to J602, R35 to R601, R36 to R602, R37 to R603, R38 to R604, R39 to R605, R40 to R606, R41 to R607, R42 to R608, U6 to U601
Changed lines of the file:
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@@
   (symbol (lib_id "Device:R") (at 222.25 73.66 0) (unit 1)
     (in_bom yes) (on_board yes) (dnp no)
-    (property "Reference" "R42" (at 220.98 68.58 0)
+    (property "Reference" "R608" (at 220.98 68.58 0)
       (effects (font (size 1.27 1.27)) (justify left))
     )
@@
       (project "SOC DISPLAY"
         (path "/9f7696f8-e9fa-4362-b2ca-5dde3355ad01/5b884267-8592-446c-85d7-63f10c8d8fbb"
-          (reference "R42") (unit 1)
+          (reference "R608") (unit 1)
         )
       )
@@
       (project "SOC DISPLAY"
         (path "/9f7696f8-e9fa-4362-b2ca-5dde3355ad01/5b884267-8592-446c-85d7-63f10c8d8fbb"
-          (reference "#PWR031") (unit 1)
+          (reference "#PWR0605") (unit 1)
         )
       )
@@
       (project "SOC DISPLAY"
         (path "/9f7696f8-e9fa-4362-b2ca-5dde3355ad01/5b884267-8592-446c-85d7-63f10c8d8fbb"
-          (reference "#PWR027") (unit 1)
+          (reference "#PWR0601") (unit 1)
         )
       )
@@
       (project "SOC DISPLAY"
         (path "/9f7696f8-e9fa-4362-b2ca-5dde3355ad01/5b884267-8592-446c-85d7-63f10c8d8fbb"
-          (reference "#PWR029") (unit 1)
+          (reference "#PWR0603") (unit 1)
         )
       )
@@
   (symbol (lib_id "Device:R") (at 113.03 67.31 90) (unit 1)
     (in_bom yes) (on_board yes) (dnp no)
-    (property "Reference" "R35" (at 113.03 64.77 90)
+    (property "Reference" "R601" (at 113.03 64.77 90)
       (effects (font (size 1.27 1.27)))
     )
@@
       (project "SOC DISPLAY"
         (path "/9f7696f8-e9fa-4362-b2ca-5dde3355ad01/5b884267-8592-446c-85d7-63f10c8d8fbb"
-          (reference "R35") (unit 1)
+          (reference "R601") (unit 1)
         )
       )
@@
   (symbol (lib_id "Device:C") (at 175.26 76.2 0) (unit 1)
     (in_bom yes) (on_board yes) (dnp no)
-    (property "Reference" "C16" (at 177.8 73.66 0)
+    (property "Reference" "C603" (at 177.8 73.66 0)
       (effects (font (size 1.27 1.27)) (justify left))
     )
@@
       (project "SOC DISPLAY"
         (path "/9f7696f8-e9fa-4362-b2ca-5dde3355ad01/5b884267-8592-446c-85d7-63f10c8d8fbb"
-          (reference "C16") (unit 1)
+          (reference "C603") (unit 1)
         )
       )
@@
   (symbol (lib_id "Device:R") (at 218.44 73.66 0) (unit 1)
     (in_bom yes) (on_board yes) (dnp no)
-    (property "Reference" "R41" (at 215.9 87.63 0)
+    (property "Reference" "R607" (at 215.9 87.63 0)
       (effects (font (size 1.27 1.27)) (justify left))
     )
@@
       (project "SOC DISPLAY"
         (path "/9f7696f8-e9fa-4362-b2ca-5dde3355ad01/5b884267-8592-446c-85d7-63f10c8d8fbb"
-          (reference "R41") (unit 1)
+          (reference "R607") (unit 1)
         )
       )
@@
   (symbol (lib_id "Device:C") (at 208.28 77.47 0) (unit 1)
     (in_bom yes) (on_board yes) (dnp no)
-    (property "Reference" "C17" (at 203.2 74.93 0)
+    (property "Reference" "C604" (at 203.2 74.93 0)
       (effects (font (size 1.27 1.27)) (justify left))
     )
@@
       (project "SOC DISPLAY"
         (path "/9f7696f8-e9fa-4362-b2ca-5dde3355ad01/5b884267-8592-446c-85d7-63f10c8d8fbb"
-          (reference "C17") (unit 1)
+          (reference "C604") (unit 1)
         )
       )
@@
   (symbol (lib_id "Device:C") (at 96.52 81.28 0) (unit 1)
     (in_bom yes) (on_board yes) (dnp no) (fields_autoplaced)
-    (property "Reference" "C15" (at 100.33 80.01 0)
+    (property "Reference" "C602" (at 100.33 80.01 0)
       (effects (font (size 1.27 1.27)) (justify left))
     )
@@
       (project "SOC DISPLAY"
         (path "/9f7696f8-e9fa-4362-b2ca-5dde3355ad01/5b884267-8592-446c-85d7-63f10c8d8fbb"
-          (reference "C15") (unit 1)
+          (reference "C602") (unit 1)
         )
       )
@@
       (project "SOC DISPLAY"
         (path "/9f7696f8-e9fa-4362-b2ca-5dde3355ad01/5b884267-8592-446c-85d7-63f10c8d8fbb"
-          (reference "#PWR033") (unit 1)
+          (reference "#PWR0607") (unit 1)
         )
       )
@@
   (symbol (lib_id "Device:R") (at 214.63 73.66 0) (unit 1)
     (in_bom yes) (on_board yes) (dnp no)
-    (property "Reference" "R40" (at 210.82 68.58 0)
+    (property "Reference" "R606" (at 210.82 68.58 0)
       (effects (font (size 1.27 1.27)) (justify left))
     )
@@
       (project "SOC DISPLAY"
         (path "/9f7696f8-e9fa-4362-b2ca-5dde3355ad01/5b884267-8592-446c-85d7-63f10c8d8fbb"
-          (reference "R40") (unit 1)
+          (reference "R606") (unit 1)
         )
       )
@@
       (project "SOC DISPLAY"
         (path "/9f7696f8-e9fa-4362-b2ca-5dde3355ad01/5b884267-8592-446c-85d7-63f10c8d8fbb"
-          (reference "#PWR032") (unit 1)
+          (reference "#PWR0606") (unit 1)
         )
       )
@@
   (symbol (lib_id "Device:R") (at 113.03 72.39 90) (unit 1)
     (in_bom yes) (on_board yes) (dnp no)
-    (property "Reference" "R36" (at 113.03 69.85 90)
+    (property "Reference" "R602" (at 113.03 69.85 90)
       (effects (font (size 1.27 1.27)))
     )
@@
       (project "SOC DISPLAY"
         (path "/9f7696f8-e9fa-4362-b2ca-5dde3355ad01/5b884267-8592-446c-85d7-63f10c8d8fbb"
-          (reference "R36") (unit 1)
+          (reference "R602") (unit 1)
         )
       )
@@
       (project "SOC DISPLAY"
         (path "/9f7696f8-e9fa-4362-b2ca-5dde3355ad01/5b884267-8592-446c-85d7-63f10c8d8fbb"
-          (reference "#PWR030") (unit 1)
+          (reference "#PWR0604") (unit 1)
         )
       )
@@
   (symbol (lib_id "Device:R") (at 181.61 68.58 90) (unit 1)
     (in_bom yes) (on_board yes) (dnp no)
-    (property "Reference" "R37" (at 181.61 66.04 90)
+    (property "Reference" "R603" (at 181.61 66.04 90)
       (effects (font (size 1.27 1.27)))
     )
@@
       (project "SOC DISPLAY"
         (path "/9f7696f8-e9fa-4362-b2ca-5dde3355ad01/5b884267-8592-446c-85d7-63f10c8d8fbb"
-          (reference "R37") (unit 1)
+          (reference "R603") (unit 1)
         )
       )
@@
   (symbol (lib_id "Connector:Conn_01x02_Pin") (at 138.43 60.96 0) (unit 1)
     (in_bom yes) (on_board yes) (dnp no) (fields_autoplaced)
-    (property "Reference" "J6" (at 139.065 55.88 0)
+    (property "Reference" "J601" (at 139.065 55.88 0)
       (effects (font (size 1.27 1.27)))
     )
@@
       (project "SOC DISPLAY"
         (path "/9f7696f8-e9fa-4362-b2ca-5dde3355ad01/5b884267-8592-446c-85d7-63f10c8d8fbb"
-          (reference "J6") (unit 1)
+          (reference "J601") (unit 1)
         )
       )
@@
   (symbol (lib_id "Device:R") (at 182.88 85.09 90) (unit 1)
     (in_bom yes) (on_board yes) (dnp no)
-    (property "Reference" "R39" (at 182.88 82.55 90)
+    (property "Reference" "R605" (at 182.88 82.55 90)
       (effects (font (size 1.27 1.27)))
     )
@@
       (project "SOC DISPLAY"
         (path "/9f7696f8-e9fa-4362-b2ca-5dde3355ad01/5b884267-8592-446c-85d7-63f10c8d8fbb"
-          (reference "R39") (unit 1)
+          (reference "R605") (unit 1)
         )
       )
@@
       (project "SOC DISPLAY"
         (path "/9f7696f8-e9fa-4362-b2ca-5dde3355ad01/5b884267-8592-446c-85d7-63f10c8d8fbb"
-          (reference "#PWR028") (unit 1)
+          (reference "#PWR0602") (unit 1)
         )
       )
@@
   (symbol (lib_id "Device:R") (at 181.61 97.79 90) (unit 1)
     (in_bom yes) (on_board yes) (dnp no)
-    (property "Reference" "R38" (at 181.61 95.25 90)
+    (property "Reference" "R604" (at 181.61 95.25 90)
       (effects (font (size 1.27 1.27)))
     )
@@
       (project "SOC DISPLAY"
         (path "/9f7696f8-e9fa-4362-b2ca-5dde3355ad01/5b884267-8592-446c-85d7-63f10c8d8fbb"
-          (reference "R38") (unit 1)
+          (reference "R604") (unit 1)
         )
       )
@@
   (symbol (lib_id "Connector:Conn_01x02_Pin") (at 157.48 59.69 0) (unit 1)
     (in_bom yes) (on_board yes) (dnp no) (fields_autoplaced)
-    (property "Reference" "J7" (at 158.115 54.61 0)
+    (property "Reference" "J602" (at 158.115 54.61 0)
       (effects (font (size 1.27 1.27)))
     )
@@
       (project "SOC DISPLAY"
         (path "/9f7696f8-e9fa-4362-b2ca-5dde3355ad01/5b884267-8592-446c-85d7-63f10c8d8fbb"
-          (reference "J7") (unit 1)
+          (reference "J602") (unit 1)
         )
       )
@@
   (symbol (lib_id "2023-08-04_10-34-25:INA228AQDGSRQ1") (at 116.84 81.28 0) (unit 1)
     (in_bom yes) (on_board yes) (dnp no) (fields_autoplaced)
-    (property "Reference" "U6" (at 137.16 71.12 0)
+    (property "Reference" "U601" (at 137.16 71.12 0)
       (effects (font (size 1.524 1.524)))
     )
@@
       (project "SOC DISPLAY"
         (path "/9f7696f8-e9fa-4362-b2ca-5dde3355ad01/5b884267-8592-446c-85d7-63f10c8d8fbb"
-          (reference "U6") (unit 1)
+          (reference "U601") (unit 1)
         )
       )
@@
   (symbol (lib_id "Device:C") (at 87.63 81.28 0) (unit 1)
     (in_bom yes) (on_board yes) (dnp no)
-    (property "Reference" "C14" (at 80.01 78.74 0)
+    (property "Reference" "C601" (at 80.01 78.74 0)
       (effects (font (size 1.27 1.27)) (justify left))
     )
@@
       (project "SOC DISPLAY"
         (path "/9f7696f8-e9fa-4362-b2ca-5dde3355ad01/5b884267-8592-446c-85d7-63f10c8d8fbb"
-          (reference "C14") (unit 1)
-        )
-      )
+          (reference "C601") (unit 1)
+        )
+      )
