File: _autosave-SOC DISPLAY.kicad_pcb (KiCad board)
At the start: 2 copper layers, 44.7 x 50.3 mm, 87 parts, among them IC1 LM5164QDDATQ1, IC2 CM BLE, J1 PRG, J2 Conn_01x05_Socket, J3 OLED, J4 OLED, J5 Conn_01x02_Socket, J6 Conn_01x02_Pin, J7 Conn_01x02_Pin, Q1 NDT3055L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

Commit message: pull
Parts:
- moved H5 4.57 mm to (76.7, 62.2)
Other:
- board size 44.7 x 50.3 mm -> 50.3 x 50.3 mm
Changed lines of the file:
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@@
   )
   (footprint "MountingHole:MountingHole_2.7mm_M2.5_ISO7380_Pad_TopBottom" (layer "F.Cu")
-    (at 72.136 62.23)
+    (at 76.708 62.23)
     (descr "Mounting Hole 2.7mm, M2.5, ISO7380")
     (tags "mounting hole 2.7mm m2.5 iso7380")
@@
     (pad "1" connect circle (at 0 0) (size 4.5 4.5) (layers "B.Cu" "B.Mask"))
   )
-  (gr_rect (start 30.099 33.02) (end 74.803 83.312)
+  (gr_rect (start 30.099 33.02) (end 80.391 83.312)
     (stroke (width 0.05) (type default)) (fill none) (layer "Edge.Cuts"))
 )
